File: NUCLEO144_wing/NUCLEO144_wing.kicad_pcb (KiCad board)
At the start: 2 copper layers, 100 x 100 mm, 14 parts, among them J1 Conn_02x36_Top_Bottom, J2 Conn_02x36_Top_Bottom, J3 Conn_02x36_Top_Bottom, J4 Conn_02x36_Top_Bottom

Commit message: to fab shop!
Parts:
- removed REF** (x2): 1pin, Connectors:1pin
- J10, J5, J6, J7, J8, J9: renamed from REF**; value rusEfi_4x39_Pitch2.54mm -> Conn_01x39
- J29, J30: renamed from REF**; value 1pin -> Conn_01x01
Connections:
- J1 pad 18: Net-(J1-Pad18) -> /5v
- J1 pad 71: Net-(J1-Pad71) -> /GND
- J1 pad 72: Net-(J1-Pad72) -> /GND
- J1 pad 8: Net-(J1-Pad8) -> /GND
- J10 pad 1: (no net) -> /GND
- J10 pad 10: (no net) -> Net-(J10-Pad10)
- J10 pad 11: (no net) -> Net-(J10-Pad11)
- J10 pad 12: (no net) -> Net-(J10-Pad12)
- J10 pad 13: (no net) -> Net-(J10-Pad13)
- J10 pad 14: (no net) -> Net-(J10-Pad14)
- J10 pad 15: (no net) -> Net-(J10-Pad15)
- J10 pad 16: (no net) -> Net-(J10-Pad16)
- J10 pad 17: (no net) -> Net-(J10-Pad17)
- J10 pad 18: (no net) -> Net-(J10-Pad18)
- J10 pad 19: (no net) -> Net-(J10-Pad19)
- J10 pad 2: (no net) -> /5v
- J10 pad 20: (no net) -> Net-(J10-Pad20)
- J10 pad 21: (no net) -> Net-(J10-Pad21)
- J10 pad 22: (no net) -> Net-(J10-Pad22)
- J10 pad 23: (no net) -> Net-(J10-Pad23)
- J10 pad 24: (no net) -> Net-(J10-Pad24)
- J10 pad 25: (no net) -> Net-(J10-Pad25)
- J10 pad 26: (no net) -> Net-(J10-Pad26)
- J10 pad 27: (no net) -> Net-(J10-Pad27)
- J10 pad 28: (no net) -> Net-(J10-Pad28)
- J10 pad 29: (no net) -> Net-(J10-Pad29)
- J10 pad 3: (no net) -> Net-(J10-Pad3)
- J10 pad 30: (no net) -> Net-(J10-Pad30)
- J10 pad 31: (no net) -> Net-(J10-Pad31)
- J10 pad 32: (no net) -> Net-(J10-Pad32)
- J10 pad 33: (no net) -> Net-(J10-Pad33)
- J10 pad 34: (no net) -> Net-(J10-Pad34)
- J10 pad 35: (no net) -> Net-(J10-Pad35)
- J10 pad 36: (no net) -> Net-(J10-Pad36)
- J10 pad 37: (no net) -> Net-(J10-Pad37)
- J10 pad 38: (no net) -> /5v
- J10 pad 39: (no net) -> /GND
- J10 pad 4: (no net) -> Net-(J10-Pad4)
- J10 pad 5: (no net) -> Net-(J10-Pad5)
- J10 pad 6: (no net) -> Net-(J10-Pad6)
- J10 pad 7: (no net) -> Net-(J10-Pad7)
- J10 pad 8: (no net) -> Net-(J10-Pad8)
- J10 pad 9: (no net) -> Net-(J10-Pad9)
- J2 pad 18: Net-(J1-Pad18) -> /5v
- J2 pad 71: Net-(J1-Pad71) -> /GND
- J2 pad 72: Net-(J1-Pad72) -> /GND
- J2 pad 8: Net-(J1-Pad8) -> /GND
- J29 pad 1: (no net) -> Net-(J29-Pad1)
- J3 pad 71: Net-(J3-Pad71) -> /GND
- J3 pad 72: Net-(J3-Pad72) -> /GND
- J30 pad 1: (no net) -> Net-(J30-Pad1)
- J4 pad 71: Net-(J3-Pad71) -> /GND
- J4 pad 72: Net-(J3-Pad72) -> /GND
- J5 pad 1: (no net) -> /GND
- J5 pad 10: (no net) -> Net-(J5-Pad10)
- J5 pad 11: (no net) -> Net-(J5-Pad11)
- J5 pad 12: (no net) -> Net-(J5-Pad12)
- J5 pad 13: (no net) -> Net-(J5-Pad13)
- J5 pad 14: (no net) -> Net-(J5-Pad14)
- J5 pad 15: (no net) -> Net-(J5-Pad15)
- J5 pad 16: (no net) -> Net-(J5-Pad16)
- J5 pad 17: (no net) -> Net-(J5-Pad17)
- J5 pad 18: (no net) -> Net-(J5-Pad18)
- J5 pad 19: (no net) -> Net-(J5-Pad19)
- J5 pad 2: (no net) -> /5v
- J5 pad 20: (no net) -> Net-(J5-Pad20)
- J5 pad 21: (no net) -> Net-(J5-Pad21)
- J5 pad 22: (no net) -> Net-(J5-Pad22)
- J5 pad 23: (no net) -> Net-(J5-Pad23)
- J5 pad 24: (no net) -> Net-(J5-Pad24)
- J5 pad 25: (no net) -> Net-(J5-Pad25)
- J5 pad 26: (no net) -> Net-(J5-Pad26)
- J5 pad 27: (no net) -> Net-(J5-Pad27)
- J5 pad 28: (no net) -> Net-(J5-Pad28)
- J5 pad 29: (no net) -> Net-(J5-Pad29)
- J5 pad 3: (no net) -> Net-(J5-Pad3)
- J5 pad 30: (no net) -> Net-(J5-Pad30)
- J5 pad 31: (no net) -> Net-(J5-Pad31)
- J5 pad 32: (no net) -> Net-(J5-Pad32)
- J5 pad 33: (no net) -> Net-(J5-Pad33)
- J5 pad 34: (no net) -> Net-(J5-Pad34)
- J5 pad 35: (no net) -> Net-(J5-Pad35)
- J5 pad 36: (no net) -> Net-(J5-Pad36)
- J5 pad 37: (no net) -> Net-(J5-Pad37)
- J5 pad 38: (no net) -> /5v
- J5 pad 39: (no net) -> /GND
- J5 pad 4: (no net) -> Net-(J5-Pad4)
- J5 pad 5: (no net) -> Net-(J5-Pad5)
- J5 pad 6: (no net) -> Net-(J5-Pad6)
- J5 pad 7: (no net) -> Net-(J5-Pad7)
- J5 pad 8: (no net) -> Net-(J5-Pad8)
- J5 pad 9: (no net) -> Net-(J5-Pad9)
- J6 pad 1: (no net) -> /GND
- J6 pad 10: (no net) -> Net-(J6-Pad10)
- J6 pad 11: (no net) -> Net-(J6-Pad11)
- J6 pad 12: (no net) -> Net-(J6-Pad12)
- J6 pad 13: (no net) -> Net-(J6-Pad13)
- J6 pad 14: (no net) -> Net-(J6-Pad14)
- J6 pad 15: (no net) -> Net-(J6-Pad15)
- J6 pad 16: (no net) -> Net-(J6-Pad16)
- J6 pad 17: (no net) -> Net-(J6-Pad17)
- J6 pad 18: (no net) -> Net-(J6-Pad18)
- J6 pad 19: (no net) -> Net-(J6-Pad19)
- J6 pad 2: (no net) -> /5v
- J6 pad 20: (no net) -> Net-(J6-Pad20)
- J6 pad 21: (no net) -> Net-(J6-Pad21)
- J6 pad 22: (no net) -> Net-(J6-Pad22)
- J6 pad 23: (no net) -> Net-(J6-Pad23)
- J6 pad 24: (no net) -> Net-(J6-Pad24)
- J6 pad 25: (no net) -> Net-(J6-Pad25)
- J6 pad 26: (no net) -> Net-(J6-Pad26)
- J6 pad 27: (no net) -> Net-(J6-Pad27)
- J6 pad 28: (no net) -> Net-(J6-Pad28)
- J6 pad 29: (no net) -> Net-(J6-Pad29)
- J6 pad 3: (no net) -> Net-(J6-Pad3)
- J6 pad 30: (no net) -> Net-(J6-Pad30)
- J6 pad 31: (no net) -> Net-(J6-Pad31)
- J6 pad 32: (no net) -> Net-(J6-Pad32)
- J6 pad 33: (no net) -> Net-(J6-Pad33)
- J6 pad 34: (no net) -> Net-(J6-Pad34)
- J6 pad 35: (no net) -> Net-(J6-Pad35)
- J6 pad 36: (no net) -> Net-(J6-Pad36)
- J6 pad 37: (no net) -> Net-(J6-Pad37)
- J6 pad 38: (no net) -> /5v
- J6 pad 39: (no net) -> /GND
- J6 pad 4: (no net) -> Net-(J6-Pad4)
- J6 pad 5: (no net) -> Net-(J6-Pad5)
- J6 pad 6: (no net) -> Net-(J6-Pad6)
- J6 pad 7: (no net) -> Net-(J6-Pad7)
- J6 pad 8: (no net) -> Net-(J6-Pad8)
- J6 pad 9: (no net) -> Net-(J6-Pad9)
- J7 pad 1: (no net) -> /GND
- J7 pad 10: (no net) -> Net-(J7-Pad10)
- J7 pad 11: (no net) -> Net-(J7-Pad11)
- J7 pad 12: (no net) -> Net-(J7-Pad12)
- J7 pad 13: (no net) -> Net-(J7-Pad13)
- J7 pad 14: (no net) -> Net-(J7-Pad14)
- J7 pad 15: (no net) -> Net-(J7-Pad15)
- J7 pad 16: (no net) -> Net-(J7-Pad16)
- J7 pad 17: (no net) -> Net-(J7-Pad17)
- J7 pad 18: (no net) -> Net-(J7-Pad18)
- J7 pad 19: (no net) -> Net-(J7-Pad19)
- J7 pad 2: (no net) -> /5v
- J7 pad 20: (no net) -> Net-(J7-Pad20)
- J7 pad 21: (no net) -> Net-(J7-Pad21)
- J7 pad 22: (no net) -> Net-(J7-Pad22)
- J7 pad 23: (no net) -> Net-(J7-Pad23)
- J7 pad 24: (no net) -> Net-(J7-Pad24)
- J7 pad 25: (no net) -> Net-(J7-Pad25)
- J7 pad 26: (no net) -> Net-(J7-Pad26)
- J7 pad 27: (no net) -> Net-(J7-Pad27)
- J7 pad 28: (no net) -> Net-(J7-Pad28)
- J7 pad 29: (no net) -> Net-(J7-Pad29)
- J7 pad 3: (no net) -> Net-(J7-Pad3)
- J7 pad 30: (no net) -> Net-(J7-Pad30)
- J7 pad 31: (no net) -> Net-(J7-Pad31)
- J7 pad 32: (no net) -> Net-(J7-Pad32)
- J7 pad 33: (no net) -> Net-(J7-Pad33)
- J7 pad 34: (no net) -> Net-(J7-Pad34)
- J7 pad 35: (no net) -> Net-(J7-Pad35)
- J7 pad 36: (no net) -> Net-(J7-Pad36)
- J7 pad 37: (no net) -> Net-(J7-Pad37)
- J7 pad 38: (no net) -> /5v
- J7 pad 39: (no net) -> /GND
- J7 pad 4: (no net) -> Net-(J7-Pad4)
- J7 pad 5: (no net) -> Net-(J7-Pad5)
- J7 pad 6: (no net) -> Net-(J7-Pad6)
- J7 pad 7: (no net) -> Net-(J7-Pad7)
- J7 pad 8: (no net) -> Net-(J7-Pad8)
- J7 pad 9: (no net) -> Net-(J7-Pad9)
- J8 pad 1: (no net) -> /GND
- J8 pad 10: (no net) -> Net-(J8-Pad10)
- J8 pad 11: (no net) -> Net-(J8-Pad11)
- J8 pad 12: (no net) -> Net-(J8-Pad12)
- J8 pad 13: (no net) -> Net-(J8-Pad13)
- J8 pad 14: (no net) -> Net-(J8-Pad14)
- J8 pad 15: (no net) -> Net-(J8-Pad15)
- J8 pad 16: (no net) -> Net-(J8-Pad16)
- J8 pad 17: (no net) -> Net-(J8-Pad17)
- J8 pad 18: (no net) -> Net-(J8-Pad18)
- J8 pad 19: (no net) -> Net-(J8-Pad19)
- J8 pad 2: (no net) -> /5v
- J8 pad 20: (no net) -> Net-(J8-Pad20)
- J8 pad 21: (no net) -> Net-(J8-Pad21)
- J8 pad 22: (no net) -> Net-(J8-Pad22)
- J8 pad 23: (no net) -> Net-(J8-Pad23)
- J8 pad 24: (no net) -> Net-(J8-Pad24)
- J8 pad 25: (no net) -> Net-(J8-Pad25)
- J8 pad 26: (no net) -> Net-(J8-Pad26)
- J8 pad 27: (no net) -> Net-(J8-Pad27)
- J8 pad 28: (no net) -> Net-(J8-Pad28)
- J8 pad 29: (no net) -> Net-(J8-Pad29)
- J8 pad 3: (no net) -> Net-(J8-Pad3)
- J8 pad 30: (no net) -> Net-(J8-Pad30)
- J8 pad 31: (no net) -> Net-(J8-Pad31)
- J8 pad 32: (no net) -> Net-(J8-Pad32)
- J8 pad 33: (no net) -> Net-(J8-Pad33)
- J8 pad 34: (no net) -> Net-(J8-Pad34)
- J8 pad 35: (no net) -> Net-(J8-Pad35)
- J8 pad 36: (no net) -> Net-(J8-Pad36)
- J8 pad 37: (no net) -> Net-(J8-Pad37)
- J8 pad 38: (no net) -> /5v
- J8 pad 39: (no net) -> /GND
- J8 pad 4: (no net) -> Net-(J8-Pad4)
- J8 pad 5: (no net) -> Net-(J8-Pad5)
- J8 pad 6: (no net) -> Net-(J8-Pad6)
- J8 pad 7: (no net) -> Net-(J8-Pad7)
- J8 pad 8: (no net) -> Net-(J8-Pad8)
- J8 pad 9: (no net) -> Net-(J8-Pad9)
- J9 pad 1: (no net) -> /GND
- J9 pad 10: (no net) -> Net-(J9-Pad10)
- J9 pad 11: (no net) -> Net-(J9-Pad11)
- J9 pad 12: (no net) -> Net-(J9-Pad12)
- J9 pad 13: (no net) -> Net-(J9-Pad13)
- J9 pad 14: (no net) -> Net-(J9-Pad14)
- J9 pad 15: (no net) -> Net-(J9-Pad15)
- J9 pad 16: (no net) -> Net-(J9-Pad16)
- J9 pad 17: (no net) -> Net-(J9-Pad17)
- J9 pad 18: (no net) -> Net-(J9-Pad18)
- J9 pad 19: (no net) -> Net-(J9-Pad19)
- J9 pad 2: (no net) -> /5v
- J9 pad 20: (no net) -> Net-(J9-Pad20)
- J9 pad 21: (no net) -> Net-(J9-Pad21)
- J9 pad 22: (no net) -> Net-(J9-Pad22)
- J9 pad 23: (no net) -> Net-(J9-Pad23)
- J9 pad 24: (no net) -> Net-(J9-Pad24)
- J9 pad 25: (no net) -> Net-(J9-Pad25)
- J9 pad 26: (no net) -> Net-(J9-Pad26)
- J9 pad 27: (no net) -> Net-(J9-Pad27)
- J9 pad 28: (no net) -> Net-(J9-Pad28)
- J9 pad 29: (no net) -> Net-(J9-Pad29)
- J9 pad 3: (no net) -> Net-(J9-Pad3)
- J9 pad 30: (no net) -> Net-(J9-Pad30)
- J9 pad 31: (no net) -> Net-(J9-Pad31)
- J9 pad 32: (no net) -> Net-(J9-Pad32)
- J9 pad 33: (no net) -> Net-(J9-Pad33)
- J9 pad 34: (no net) -> Net-(J9-Pad34)
- J9 pad 35: (no net) -> Net-(J9-Pad35)
- J9 pad 36: (no net) -> Net-(J9-Pad36)
- J9 pad 37: (no net) -> Net-(J9-Pad37)
- J9 pad 38: (no net) -> /5v
- J9 pad 39: (no net) -> /GND
- J9 pad 4: (no net) -> Net-(J9-Pad4)
- J9 pad 5: (no net) -> Net-(J9-Pad5)
- J9 pad 6: (no net) -> Net-(J9-Pad6)
- J9 pad 7: (no net) -> Net-(J9-Pad7)
- J9 pad 8: (no net) -> Net-(J9-Pad8)
- J9 pad 9: (no net) -> Net-(J9-Pad9)
Routing:
- net Net-(J1-Pad18): track 231.9 -> 0.00 mm
- net /5v: track 0.00 -> 231.9 mm
- net /GND: track 0.00 -> 166.4 mm
- net Net-(J1-Pad71): track 88.5 -> 0.00 mm
- net Net-(J1-Pad8): track 30.9 -> 0.00 mm
- net Net-(J3-Pad72): track 20.6 -> 0.00 mm
- net Net-(J3-Pad71): track 15.2 -> 0.00 mm
- net Net-(J1-Pad72): track 11.2 -> 0.00 mm
- added copper zone on B.Cu, net /5v
- added copper zone on F.Cu, net /GND
- removed copper zone on B.Cu, net GND
- removed copper zone on F.Cu, net GND
