File: NUCLEO144_wing/NUCLEO144_wing.sch (KiCad schematic (older format))
At the start: 7 parts, among them J1 Conn_02x36_Top_Bottom, J2 Conn_02x36_Top_Bottom, J20 Conn_02x40_Odd_Even, J3 Conn_02x36_Top_Bottom, J4 Conn_02x36_Top_Bottom, U1 NUCLEO144-F429ZI, U2 NUCLEO144-F429ZI

Commit message: to fab shop!
Parts:
- removed J20: Conn_02x40_Odd_Even, symbol Conn_02x40_Odd_Even
- removed U1, U2: NUCLEO144-F429ZI, rusEFI_LIB:ST_Morpho_Connector_144_STLink, symbol NUCLEO144-F429ZI
- added J10, J5, J6, J7, J8, J9: Conn_01x39, rusEFI_local:rusEfi_4x39_Pitch2.54mm, symbol Conn_01x39
- added J29, J30: Conn_01x01, Connectors:1pin, symbol Conn_01x01
Connections:
- net labels added: 5v, GND
- wire segments 240 -> 224
Other:
- moved on the sheet: J3, J4
