File: highside_module/hi-lo.kicad_pcb (KiCad board)
At the start: 2 copper layers, 43.4 x 20.3 mm, 30 parts, among them M601 CONN_1, P601 CONN_3X2, P602 CONN_2, P603 CONN_6, P604 CONN_2, U601 TC4427, U602 TC4427, U603 TC4427

Commit message: gerbers
Other:
- board text added: "R0.3 rusefi.com"
- board text removed: "R.03 rusefi.com"
Changed lines of the file:
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@@
     (links 51)
     (no_connects 0)
-    (area 28.778999 12.121499 224.790001 255.053501)
+    (area 28.778999 12.121499 247.169715 255.053501)
     (thickness 1.6)
-    (drawings 47)
+    (drawings 51)
     (tracks 301)
     (zones 0)
@@
   (title_block
     (title "High or low side drive board for RUSEFI.com")
-    (rev .01)
+    (rev 0.3)
     (company RUSEFI.com)
     (comment 2 Art_Electro)
@@
     )
   )
+  (dimension 20.32 (width 0.3) (layer Cmts.User)
+    (gr_text "0.8000 in" (at 241.634 158.75 270) (layer Cmts.User)
+      (effects (font (size 1.5 1.5) (thickness 0.3)))
+    )
+    (feature1 (pts (xy 237.236 168.91) (xy 242.984 168.91)))
+    (feature2 (pts (xy 237.236 148.59) (xy 242.984 148.59)))
+    (crossbar (pts (xy 240.284 148.59) (xy 240.284 168.91)))
+    (arrow1a (pts (xy 240.284 168.91) (xy 239.697579 167.783496)))
+    (arrow1b (pts (xy 240.284 168.91) (xy 240.870421 167.783496)))
+    (arrow2a (pts (xy 240.284 148.59) (xy 239.697579 149.716504)))
+    (arrow2b (pts (xy 240.284 148.59) (xy 240.870421 149.716504)))
+  )
+  (dimension 43.688738 (width 0.3) (layer Cmts.User)
+    (gr_text "1.7200 in" (at 196.862252 133.14748 359.6668888) (layer Cmts.User)
+      (effects (font (size 1.5 1.5) (thickness 0.3)))
+    )
+    (feature1 (pts (xy 218.694 135.382) (xy 218.714101 131.924503)))
+    (feature2 (pts (xy 175.006 135.128) (xy 175.026101 131.670503)))
+    (crossbar (pts (xy 175.010404 134.370457) (xy 218.698404 134.624457)))
+    (arrow1a (pts (xy 218.698404 134.624457) (xy 217.56851 135.204318)))
+    (arrow1b (pts (xy 218.698404 134.624457) (xy 217.575329 134.031497)))
+    (arrow2a (pts (xy 175.010404 134.370457) (xy 176.133479 134.963417)))
+    (arrow2b (pts (xy 175.010404 134.370457) (xy 176.140298 133.790596)))
+  )
+  (dimension 20.326349 (width 0.3) (layer Cmts.User)
+    (gr_text "20.326 mm" (at 232.994087 158.669352 88.56790382) (layer Cmts.User)
+      (effects (font (size 1.5 1.5) (thickness 0.3)))
+    )
+    (feature1 (pts (xy 225.806 168.656) (xy 234.089666 168.863092)))
+    (feature2 (pts (xy 226.314 148.336) (xy 234.597666 148.543092)))
+    (crossbar (pts (xy 231.898509 148.475613) (xy 231.390509 168.795613)))
+    (arrow1a (pts (xy 231.390509 168.795613) (xy 230.832425 167.654805)))
+    (arrow1b (pts (xy 231.390509 168.795613) (xy 232.0049 167.684117)))
+    (arrow2a (pts (xy 231.898509 148.475613) (xy 231.284118 149.587109)))
+    (arrow2b (pts (xy 231.898509 148.475613) (xy 232.456593 149.616421)))
+  )
+  (dimension 43.434743 (width 0.3) (layer Cmts.User)
+    (gr_text "43.435 mm" (at 196.744253 140.510587 359.6649408) (layer Cmts.User)
+      (effects (font (size 1.5 1.5) (thickness 0.3)))
+    )
+    (feature1 (pts (xy 218.44 144.272) (xy 218.469148 139.28761)))
+    (feature2 (pts (xy 175.006 144.018) (xy 175.035148 139.03361)))
+    (crossbar (pts (xy 175.019359 141.733564) (xy 218.453359 141.987564)))
+    (arrow1a (pts (xy 218.453359 141.987564) (xy 217.323445 142.567387)))
+    (arrow1b (pts (xy 218.453359 141.987564) (xy 217.330304 141.394566)))
+    (arrow2a (pts (xy 175.019359 141.733564) (xy 176.142414 142.326562)))
+    (arrow2b (pts (xy 175.019359 141.733564) (xy 176.149273 141.153741)))
+  )
   (gr_text P203 (at 213.868 156.337) (layer B.SilkS)
     (effects (font (size 1.016 1.016) (thickness 0.2032)) (justify mirror))
@@
   (gr_line (start 209.55 151.765) (end 209.55 149.86) (angle 90) (layer B.SilkS) (width 0.1))
   (gr_line (start 209.55 151.13) (end 209.55 151.765) (angle 90) (layer B.SilkS) (width 0.1))
-  (gr_text "R.03\nrusefi.com" (at 183.896 157.988) (layer B.SilkS)
+  (gr_text "R0.3\nrusefi.com" (at 183.896 157.988) (layer B.SilkS)
     (effects (font (size 1.016 1.016) (thickness 0.2032)) (justify left mirror))
   )

Commit message: progress
Parts:
- added P606: CONN_2, SIL-2, F.Cu at (179.1, 165.1)
- moved P604 10.2 mm to (179.1, 162.6)
- moved M601 7.19 mm to (178.3, 152.1)
Routing:
- net /VP: track 42.1 -> 66.7 mm
- net GND: track 132.2 -> 136.4 mm, vias 31 -> 32
- net 5V: track 0.00 -> 2.54 mm
- net /H_IN1: track 32.2 -> 34.5 mm
- net /HL1: track 43.2 -> 44.6 mm
- net /H_IN2: track 12.8 -> 12.1 mm
- net /HL3: track 32.3 -> 32.6 mm, vias 2 -> 4

Commit message: silkscreen
Other:
- board text added: "O1"
- board text added: "O2"
- board text added: "O3"
- board text added: "O4"
- board text added: "O5"
- board text added: "O6"
Changed lines of the file:
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@@
-(kicad_pcb (version 4) (host pcbnew 4.0.7)
+(kicad_pcb (version 4) (host pcbnew 4.0.1-stable)
   (general
     (links 53)
     (no_connects 0)
-    (area 28.778999 12.121499 247.169715 255.053501)
+    (area 28.778999 12.121499 247.319715 255.053501)
     (thickness 1.6)
-    (drawings 51)
+    (drawings 57)
     (tracks 317)
     (zones 0)
@@
     )
   )
+  (gr_text O5 (at 195.326 162.814) (layer F.Cu)
+    (effects (font (size 1.2 1.2) (thickness 0.3)))
+  )
+  (gr_text O6 (at 193.04 162.814) (layer F.Cu)
+    (effects (font (size 1.2 1.2) (thickness 0.3)))
+  )
+  (gr_text O4 (at 190.5 162.814) (layer F.Cu)
+    (effects (font (size 1.2 1.2) (thickness 0.3)))
+  )
+  (gr_text O3 (at 182.88 162.814) (layer F.Cu)
+    (effects (font (size 1.2 1.2) (thickness 0.3)))
+  )
+  (gr_text O2 (at 187.96 162.814) (layer F.Cu)
+    (effects (font (size 1.2 1.2) (thickness 0.3)))
+  )
+  (gr_text O1 (at 185.674 162.814) (layer F.Cu)
+    (effects (font (size 1.2 1.2) (thickness 0.3)))
+  )
   (dimension 20.32 (width 0.3) (layer Cmts.User)
