File: TLE8888_Module/TLE8888_Module.sch (KiCad schematic (older format))
At the start: 41 parts, among them J1 Conn_01x01, J2 Conn_02x39_Odd_Even, Q1 IPD30N06S2L-23, U2 TLE8888QK

Commit message: sync
Parts:
- J2: footprint Connector_PinHeader_2.54mm:PinHeader_2x39_P2.54mm_Vertical -> Connector_PinHeader_2.54mm:Conn_TLE8888_Module
Connections:
- net 5V1: now also J2.57 (Pin_57); no longer J2.65 (Pin_65)
- net 5V2: now also J2.58 (Pin_58); no longer J2.66 (Pin_66)
- net CAN_H: no longer J2.25 (Pin_25)
- net CAN_L: no longer J2.26 (Pin_26)
- net CAN_RX: no longer J2.23 (Pin_23)
- net CAN_TX: no longer J2.24 (Pin_24)
- net CRNK+: now also J2.63 (Pin_63); no longer J2.78 (Pin_78)
- net CRNK-: now also J2.64 (Pin_64); no longer J2.77 (Pin_77)
- net CRNK_MCU: now also J2.62 (Pin_62); no longer J2.71 (Pin_71)
- net CSN: now also J2.53 (Pin_53); no longer J2.61 (Pin_61)
- net DFB_10: now also J2.31 (Pin_31); no longer J2.41 (Pin_41)
- net DFB_11: now also J2.35 (Pin_35); no longer J2.43 (Pin_43)
- net DFB_12: now also J2.42 (Pin_42); no longer J2.45 (Pin_45)
- net DFB_13: now also J2.40 (Pin_40); no longer J2.47 (Pin_47)
- net DFB_8: now also J2.30 (Pin_30); no longer J2.37 (Pin_37)
- net DFB_9: now also J2.29 (Pin_29); no longer J2.38 (Pin_38)
- net FCLP: now also J2.56 (Pin_56); no longer J2.64 (Pin_64)
- net GND: now also J2.65 (Pin_65), J2.66 (Pin_66)
- net IGN_IN_1: now also J2.12 (Pin_12); no longer J2.15 (Pin_15)
- net IGN_IN_2: now also J2.13 (Pin_13); no longer J2.16 (Pin_16)
- net IGN_IN_3: now also J2.14 (Pin_14); no longer J2.17 (Pin_17)
- net IGN_IN_4: now also J2.15 (Pin_15); no longer J2.18 (Pin_18)
- net IGN_OUT_1: now also J2.49 (Pin_49); no longer J2.57 (Pin_57)
- net IGN_OUT_2: now also J2.50 (Pin_50); no longer J2.58 (Pin_58)
- net IGN_OUT_3: now also J2.51 (Pin_51); no longer J2.59 (Pin_59)
- net IGN_OUT_4: now also J2.52 (Pin_52); no longer J2.60 (Pin_60)
- net INJ_IN_1: now also J2.8 (Pin_8); no longer J2.11 (Pin_11)
- net INJ_IN_2: now also J2.9 (Pin_9); no longer J2.12 (Pin_12)
- net INJ_IN_3: now also J2.10 (Pin_10); no longer J2.13 (Pin_13)
- net INJ_IN_4: now also J2.11 (Pin_11); no longer J2.14 (Pin_14)
- net IN_10: now also J2.17 (Pin_17); no longer J2.20 (Pin_20)
- net IN_11: now also J2.18 (Pin_18); no longer J2.21 (Pin_21)
- net IN_12: now also J2.19 (Pin_19); no longer J2.22 (Pin_22)
- net IN_9: now also J2.16 (Pin_16); no longer J2.19 (Pin_19)
- net LIN_IO: no longer J2.49 (Pin_49)
- net LIN_RX: no longer J2.73 (Pin_73)
- net LIN_TX: no longer J2.72 (Pin_72)
- net MAIN_RELAY: no longer J2.27 (Pin_27)
- net OUT_1: now also J2.24 (Pin_24); no longer J2.31 (Pin_31)
- net OUT_10: now also J2.33 (Pin_33); no longer J2.42 (Pin_42)
- net OUT_11: now also J2.37 (Pin_37); no longer J2.44 (Pin_44)
- net OUT_12: now also J2.39 (Pin_39); no longer J2.46 (Pin_46)
- net OUT_13: now also J2.41 (Pin_41); no longer J2.48 (Pin_48)
- net OUT_14: now also J2.28 (Pin_28); no longer J2.36 (Pin_36)
- net OUT_15: now also J2.27 (Pin_27); no longer J2.35 (Pin_35)
- net OUT_16: now also J2.21 (Pin_21); no longer J2.30 (Pin_30)
- net OUT_17: now also J2.22 (Pin_22); no longer J2.29 (Pin_29)
- net OUT_18: now also J2.20 (Pin_20); no longer J2.28 (Pin_28)
- net OUT_19: now also J2.61 (Pin_61); no longer J2.70 (Pin_70)
- net OUT_2: now also J2.23 (Pin_23); no longer J2.32 (Pin_32)
- net OUT_20: now also J2.60 (Pin_60); no longer J2.69 (Pin_69)
- net OUT_21: now also J2.47 (Pin_47); no longer J2.54 (Pin_54)
- net OUT_22: now also J2.46 (Pin_46); no longer J2.53 (Pin_53)
- net OUT_23: now also J2.45 (Pin_45); no longer J2.52 (Pin_52)
- net OUT_24: now also J2.48 (Pin_48); no longer J2.51 (Pin_51)
- net OUT_3: now also J2.26 (Pin_26); no longer J2.33 (Pin_33)
- net OUT_4: now also J2.25 (Pin_25); no longer J2.34 (Pin_34)
- net OUT_5: now also J2.36 (Pin_36); no longer J2.50 (Pin_50)
- net OUT_6: now also J2.38 (Pin_38); no longer J2.56 (Pin_56)
- net OUT_7: now also J2.59 (Pin_59); no longer J2.68 (Pin_68)
- net OUT_8: now also J2.34 (Pin_34); no longer J2.39 (Pin_39)
- net OUT_9: now also J2.32 (Pin_32); no longer J2.40 (Pin_40)
- net SDO: now also J2.54 (Pin_54); no longer J2.62 (Pin_62)
- net SIP: now also J2.55 (Pin_55); no longer J2.63 (Pin_63)
- net V5V: now also J2.43 (Pin_43), J2.44 (Pin_44)
- net VDD: now also J2.7 (Pin_7); no longer J2.10 (Pin_10), J2.9 (Pin_9)
Changed lines of the file:
@@
 Text Label 10650 6700 1    50   ~ 10
 MAIN_RELAY
-Text Label 4550 5150 0    50   ~ 10
+Text Label 4550 4750 0    50   ~ 10
 OUT_14
-Text Label 4050 5150 2    50   ~ 10
+Text Label 4050 4750 2    50   ~ 10
 OUT_15
-Text Label 4550 5050 0    50   ~ 10
+Text Label 4050 4650 2    50   ~ 10
 OUT_4
-Text Label 4050 5050 2    50   ~ 10
+Text Label 4550 4650 0    50   ~ 10
 OUT_3
-Text Label 4550 4950 0    50   ~ 10
+Text Label 4050 4550 2    50   ~ 10
 OUT_2
-Text Label 4050 4950 2    50   ~ 10
+Text Label 4550 4550 0    50   ~ 10
 OUT_1
-Text Label 4550 4850 0    50   ~ 10
+Text Label 4050 4450 2    50   ~ 10
 OUT_16
-Text Label 4050 4850 2    50   ~ 10
+Text Label 4550 4450 0    50   ~ 10
 OUT_17
-Text Label 4550 4750 0    50   ~ 10
+Text Label 4550 4350 0    50   ~ 10
 OUT_18
-Text Label 4050 4750 2    50   ~ 10
+Text Label 6100 6000 2    50   ~ 10
 MAIN_RELAY
 Text Label 13150 6250 0    50   ~ 10
@@
 Text Label 9150 10100 3    50   ~ 10
 FCLP
-Text Label 4550 6550 0    50   ~ 10
+Text Label 4550 6150 0    50   ~ 10
 FCLP
-Text Label 4050 6550 2    50   ~ 10
+Text Label 4050 6150 2    50   ~ 10
 SIP
-Text Label 4550 6450 0    50   ~ 10
+Text Label 4550 6050 0    50   ~ 10
 SDO
-Text Label 4050 6450 2    50   ~ 10
+Text Label 4050 6050 2    50   ~ 10
 CSN
 Text Label 9950 10100 3    50   ~ 10
-OUT_7
-Text Label 4550 6750 0    50   ~ 10
 OUT_7
 Text Label 10550 10400 0    50   ~ 10
@@
 Wire Wire Line
 	10550 10100 10550 10400
-Text Label 4050 6950 2    50   ~ 10
+Text Label 4550 6450 0    50   ~ 10
 CRNK_MCU
 Text Label 8000 11400 0    50   ~ 10
@@
 Text Label 8900 11450 0    50   ~ 0
 V5V
-Text Label 4050 6650 2    50   ~ 10
+Text Label 4050 6250 2    50   ~ 10
 5V1
-Text Label 4550 6650 0    50   ~ 10
+Text Label 4550 6250 0    50   ~ 10
 5V2
 Text Label 8750 6700 1    50   ~ 10
@@
 Text Label 9250 6700 1    50   ~ 10
 DFB_8
-Text Label 4550 5450 0    50   ~ 10
+Text Label 4050 5050 2    50   ~ 10
 OUT_10
-Text Label 4050 5450 2    50   ~ 10
+Text Label 4050 4950 2    50   ~ 10
 DFB_10
-Text Label 4550 5350 0    50   ~ 10
+Text Label 4550 4950 0    50   ~ 10
 OUT_9
-Text Label 4050 5350 2    50   ~ 10
+Text Label 4550 5050 0    50   ~ 10
 OUT_8
-Text Label 4550 5250 0    50   ~ 10
+Text Label 4050 4850 2    50   ~ 10
 DFB_9
-Text Label 4050 5250 2    50   ~ 10
+Text Label 4550 4850 0    50   ~ 10
 DFB_8
 Text Label 8100 7300 2    50   ~ 10
@@
 Text Label 8000 8200 2    50   ~ 10
 OUT_24
-Text Label 4550 5550 0    50   ~ 10
+Text Label 4050 5250 2    50   ~ 10
 OUT_11
-Text Label 4550 5650 0    50   ~ 10
+Text Label 4050 5350 2    50   ~ 10
 OUT_12
+Text Label 4050 5450 2    50   ~ 10
+OUT_13
+Text Label 4050 5150 2    50   ~ 10
+DFB_11
+Text Label 4550 5450 0    50   ~ 10
+DFB_12
+Text Label 4550 5350 0    50   ~ 10
+DFB_13
+Text Label 4550 5150 0    50   ~ 10
+OUT_5
 Text Label 4550 5750 0    50   ~ 10
-OUT_13
-Text Label 4050 5550 2    50   ~ 10
-DFB_11
-Text Label 4050 5650 2    50   ~ 10
-DFB_12
-Text Label 4050 5750 2    50   ~ 10
-DFB_13
-Text Label 4550 5850 0    50   ~ 10
-OUT_5
-Text Label 4050 5950 2    50   ~ 10
 OUT_24
 Text Label 8000 8400 2    50   ~ 10
@@
 Text Label 8000 8900 2    50   ~ 10
 OUT_6
-Text Label 4550 5950 0    50   ~ 10
+Text Label 4050 5650 2    50   ~ 10
 OUT_23
-Text Label 4550 6050 0    50   ~ 10
+Text Label 4050 5750 2    50   ~ 10
 OUT_21
 Text Label 7350 9200 2    50   ~ 10
@@
 Text Label 8100 9500 2    50   ~ 10
 IGN_OUT_4
-Text Label 4050 6350 2    50   ~ 10
+Text Label 4050 5950 2    50   ~ 10
 IGN_OUT_3
-Text Label 4550 6350 0    50   ~ 10
+Text Label 4550 5950 0    50   ~ 10
 IGN_OUT_4
-Text Label 4050 6250 2    50   ~ 10
+Text Label 4050 5850 2    50   ~ 10
 IGN_OUT_1
 Text Label 10250 10450 0    50   ~ 10
@@
 Text Label 10150 10550 0    50   ~ 10
 OUT_20
-Text Label 4550 6850 0    50   ~ 10
+Text Label 4050 6450 2    50   ~ 10
 OUT_19
-Text Label 4050 6850 2    50   ~ 10
-OUT_20
 Text Label 12550 5550 0    50   ~ 10
 12V
@@
 Text Label 15050 7950 0    50   ~ 10
 CAN_H
-Text Label 4550 3550 0    60   ~ 12
+Text Label 4550 5550 0    60   ~ 12
 V5V
 $Comp
@@
 F 0 "J2" H 4300 7467 50  0000 C CNN
 F 1 "Conn_02x39_Odd_Even" H 4300 7376 50  0000 C CNN
-F 2 "Connector_PinHeader_2.54mm:PinHeader_2x39_P2.54mm_Vertical" H 4250 5350 50  0001 C CNN
+F 2 "Connector_PinHeader_2.54mm:Conn_TLE8888_Module" H 4250 5350 50  0001 C CNN
 F 3 "~" H 4250 5350 50  0001 C CNN
 	1    4250 5350
@@
 Text Label 8100 7800 2    50   ~ 0
 LIN_IO
-Text Label 4050 5850 2    50   ~ 0
+Text Label 5950 6350 2    50   ~ 0
 LIN_IO
-Text Label 4550 6150 0    50   ~ 10
+Text Label 4550 5250 0    50   ~ 10
 OUT_6
-Text Label 4550 6250 0    50   ~ 10
+Text Label 4550 5850 0    50   ~ 10
 IGN_OUT_2
-Text Label 4050 6050 2    50   ~ 10
+Text Label 4550 5650 0    50   ~ 10
 OUT_22
 Text Label 10750 10100 3    50   ~ 0
@@
 Text Label 10650 10100 3    50   ~ 0
 LIN_TX
-Text Label 4050 7050 2    50   ~ 0
+Text Label 6000 6250 2    50   ~ 0
 LIN_RX
-Text Label 4550 6950 0    50   ~ 0
+Text Label 5750 6150 0    50   ~ 0
 LIN_TX
-Text Label 4050 7250 2    50   ~ 10
-CRNK-
-Text Label 4550 7250 0    50   ~ 10
-CRNK+
+Text Label 4050 3850 2    50   ~ 10
+INJ_IN_2
+Text Label 4050 3950 2    50   ~ 10
+INJ_IN_4
+Text Label 2750 4100 2    50   ~ 10
+CAN_L
+Text Label 4050 4050 2    50   ~ 10
+IGN_IN_2
+Text Label 4050 4150 2    50   ~ 10
+IGN_IN_4
+Text Label 4050 4250 2    50   ~ 10
+IN_10
+Text Label 4050 4350 2    50   ~ 10
+IN_12
+Text Label 2750 4000 2    50   ~ 10
+CAN_TX
+Text Label 4550 3850 0    50   ~ 10
+INJ_IN_3
+Text Label 4050 3750 2    60   ~ 12
+VDD
+Text Label 3000 4100 0    50   ~ 10
+CAN_H
+Text Label 4550 3750 0    50   ~ 10
+INJ_IN_1
 Text Label 4550 3950 0    50   ~ 10
-INJ_IN_2
+IGN_IN_1
 Text Label 4550 4050 0    50   ~ 10
-INJ_IN_4
-Text Label 4550 4650 0    50   ~ 10
-CAN_L
-Text Label 4550 3850 0    60   ~ 12
-VDD
+IGN_IN_3
 Text Label 4550 4150 0    50   ~ 10
-IGN_IN_2
+IN_9
 Text Label 4550 4250 0    50   ~ 10
-IGN_IN_4
-Text Label 4550 4350 0    50   ~ 10
-IN_10
-Text Label 4550 4450 0    50   ~ 10
-IN_12
-Text Label 4550 4550 0    50   ~ 10
-CAN_TX
-Text Label 4050 4050 2    50   ~ 10
-INJ_IN_3
-Text Label 4050 3850 2    60   ~ 12
-VDD
-Text Label 4050 4650 2    50   ~ 10
-CAN_H
-Text Label 4050 3950 2    50   ~ 10
-INJ_IN_1
-Text Label 4050 4150 2    50   ~ 10
-IGN_IN_1
-Text Label 4050 4250 2    50   ~ 10
-IGN_IN_3
-Text Label 4050 4350 2    50   ~ 10
-IN_9
-Text Label 4050 4450 2    50   ~ 10
 IN_11
-Text Label 4050 4550 2    50   ~ 10
+Text Label 3000 4000 0    50   ~ 10
 CAN_RX
 Wire Wire Line
@@
 Wire Wire Line
 	12850 6550 12850 6750
+Text Label 4050 6550 2    50   ~ 10
+CRNK+
+Text Label 4550 6550 0    50   ~ 10
+CRNK-
+Text Label 4550 6350 0    50   ~ 10
+OUT_20
+Text Label 4050 6350 2    50   ~ 10
+OUT_7
+Text Label 4050 5550 2    60   ~ 12
+V5V
+Text Label 4050 6650 2    60   ~ 12
+GND
+Text Label 4550 6650 0    60   ~ 12
+GND
+Text Label 4550 3550 0    60   ~ 12
+V5V
 $EndSCHEMATC

Commit message: sync
Parts:
- added HS1, HS2: Heatsink, Heatsink:HEATSINK, symbol Mechanical:Heatsink
- added J3: Conn_02x04_Odd_Even, Connector_PinHeader_1.00mm:PinHeader_2x04_P1.00mm_Vertical, symbol Connector_Generic:Conn_02x04_Odd_Even
Connections:
- net 12V: now also J2.61 (Pin_61), J2.62 (Pin_62); no longer J2.5 (Pin_5), J2.6 (Pin_6)
- net 5V1: now also J2.53 (Pin_53); no longer J2.57 (Pin_57)
- net 5V2: now also J2.54 (Pin_54); no longer J2.58 (Pin_58)
- net CAN_H: now also J3.5 (Pin_5)
- net CAN_L: now also J3.3 (Pin_3)
- net CAN_RX: now also J3.2 (Pin_2)
- net CAN_TX: now also J3.4 (Pin_4)
- net CRNK+: now also J2.59 (Pin_59); no longer J2.63 (Pin_63)
- net CRNK-: now also J2.60 (Pin_60); no longer J2.64 (Pin_64)
- net CRNK_MCU: now also J2.58 (Pin_58); no longer J2.62 (Pin_62)
- net CSN: now also J2.49 (Pin_49); no longer J2.53 (Pin_53)
- net DFB_10: now also J2.29 (Pin_29); no longer J2.31 (Pin_31)
- net DFB_11: now also J2.33 (Pin_33); no longer J2.35 (Pin_35)
- net DFB_12: now also J2.40 (Pin_40); no longer J2.42 (Pin_42)
- net DFB_13: now also J2.38 (Pin_38); no longer J2.40 (Pin_40)
- net DFB_8: now also J2.28 (Pin_28); no longer J2.30 (Pin_30)
- net DFB_9: now also J2.27 (Pin_27); no longer J2.29 (Pin_29)
- net FCLP: now also J2.52 (Pin_52); no longer J2.56 (Pin_56)
- net IGN_IN_1: now also J2.10 (Pin_10); no longer J2.12 (Pin_12)
- net IGN_IN_2: now also J2.11 (Pin_11); no longer J2.13 (Pin_13)
- net IGN_IN_3: now also J2.12 (Pin_12); no longer J2.14 (Pin_14)
- net IGN_IN_4: now also J2.13 (Pin_13); no longer J2.15 (Pin_15)
- net IGN_OUT_1: now also J2.45 (Pin_45); no longer J2.49 (Pin_49)
- net IGN_OUT_2: now also J2.46 (Pin_46); no longer J2.50 (Pin_50)
- net IGN_OUT_3: now also J2.47 (Pin_47); no longer J2.51 (Pin_51)
- net IGN_OUT_4: now also J2.48 (Pin_48); no longer J2.52 (Pin_52)
- net INJ_IN_1: now also J2.6 (Pin_6); no longer J2.8 (Pin_8)
- net INJ_IN_2: now also J2.7 (Pin_7); no longer J2.9 (Pin_9)
- net INJ_IN_3: now also J2.8 (Pin_8); no longer J2.10 (Pin_10)
- net INJ_IN_4: now also J2.9 (Pin_9); no longer J2.11 (Pin_11)
- net IN_10: now also J2.15 (Pin_15); no longer J2.17 (Pin_17)
- net IN_11: now also J2.16 (Pin_16); no longer J2.18 (Pin_18)
- net IN_12: now also J2.17 (Pin_17); no longer J2.19 (Pin_19)
- net IN_9: now also J2.14 (Pin_14); no longer J2.16 (Pin_16)
- net LIN_IO: now also J3.7 (Pin_7)
- net LIN_RX: now also J3.6 (Pin_6)
- net LIN_TX: now also J3.8 (Pin_8)
- net MAIN_RELAY: now also J3.1 (Pin_1)
- net OUT_1: now also J2.22 (Pin_22); no longer J2.24 (Pin_24)
- net OUT_10: now also J2.31 (Pin_31); no longer J2.33 (Pin_33)
- net OUT_11: now also J2.35 (Pin_35); no longer J2.37 (Pin_37)
- net OUT_12: now also J2.37 (Pin_37); no longer J2.39 (Pin_39)
- net OUT_13: now also J2.39 (Pin_39); no longer J2.41 (Pin_41)
- net OUT_14: now also J2.26 (Pin_26); no longer J2.28 (Pin_28)
- net OUT_15: now also J2.25 (Pin_25); no longer J2.27 (Pin_27)
- net OUT_16: now also J2.19 (Pin_19); no longer J2.21 (Pin_21)
- net OUT_17: now also J2.20 (Pin_20); no longer J2.22 (Pin_22)
- net OUT_18: now also J2.18 (Pin_18); no longer J2.20 (Pin_20)
- net OUT_19: now also J2.57 (Pin_57); no longer J2.61 (Pin_61)
- net OUT_2: now also J2.21 (Pin_21); no longer J2.23 (Pin_23)
- net OUT_20: now also J2.56 (Pin_56); no longer J2.60 (Pin_60)
- net OUT_21: now also J2.43 (Pin_43); no longer J2.47 (Pin_47)
- net OUT_22: now also J2.44 (Pin_44); no longer J2.46 (Pin_46)
- net OUT_23: now also J2.42 (Pin_42); no longer J2.45 (Pin_45)
- net OUT_24: now also J2.41 (Pin_41); no longer J2.48 (Pin_48)
- net OUT_3: now also J2.24 (Pin_24); no longer J2.26 (Pin_26)
- net OUT_4: now also J2.23 (Pin_23); no longer J2.25 (Pin_25)
- net OUT_5: now also J2.34 (Pin_34); no longer J2.36 (Pin_36)
- net OUT_6: now also J2.36 (Pin_36); no longer J2.38 (Pin_38)
- net OUT_7: now also J2.55 (Pin_55); no longer J2.59 (Pin_59)
- net OUT_8: now also J2.32 (Pin_32); no longer J2.34 (Pin_34)
- net OUT_9: now also J2.30 (Pin_30); no longer J2.32 (Pin_32)
- net SDO: now also J2.50 (Pin_50); no longer J2.54 (Pin_54)
- net SIP: now also J2.51 (Pin_51); no longer J2.55 (Pin_55)
- net V5V: now also J2.63 (Pin_63), J2.64 (Pin_64); no longer J2.43 (Pin_43), J2.44 (Pin_44)
- net VDD: now also J2.5 (Pin_5); no longer J2.7 (Pin_7)
Changed lines of the file:
@@
 Text Label 10650 6700 1    50   ~ 10
 MAIN_RELAY
-Text Label 4550 4750 0    50   ~ 10
+Text Label 4550 4650 0    50   ~ 10
 OUT_14
-Text Label 4050 4750 2    50   ~ 10
+Text Label 4050 4650 2    50   ~ 10
 OUT_15
-Text Label 4050 4650 2    50   ~ 10
+Text Label 4050 4550 2    50   ~ 10
 OUT_4
-Text Label 4550 4650 0    50   ~ 10
+Text Label 4550 4550 0    50   ~ 10
 OUT_3
-Text Label 4050 4550 2    50   ~ 10
+Text Label 4050 4450 2    50   ~ 10
 OUT_2
-Text Label 4550 4550 0    50   ~ 10
+Text Label 4550 4450 0    50   ~ 10
 OUT_1
-Text Label 4050 4450 2    50   ~ 10
+Text Label 4050 4350 2    50   ~ 10
 OUT_16
-Text Label 4550 4450 0    50   ~ 10
+Text Label 4550 4350 0    50   ~ 10
 OUT_17
-Text Label 4550 4350 0    50   ~ 10
+Text Label 4550 4250 0    50   ~ 10
 OUT_18
-Text Label 6100 6000 2    50   ~ 10
+Text Label 2400 2900 2    50   ~ 10
 MAIN_RELAY
 Text Label 13150 6250 0    50   ~ 10
@@
 Text Label 5550 8600 0    50   ~ 10
 12V
-Text Label 4550 3650 0    50   ~ 10
+Text Label 4550 6450 0    50   ~ 10
 12V
 Text Label 8750 10100 3    50   ~ 10
@@
 Text Label 9150 10100 3    50   ~ 10
 FCLP
-Text Label 4550 6150 0    50   ~ 10
-FCLP
-Text Label 4050 6150 2    50   ~ 10
+Text Label 4050 5950 2    50   ~ 10
 SIP
-Text Label 4550 6050 0    50   ~ 10
-SDO
-Text Label 4050 6050 2    50   ~ 10
-CSN
 Text Label 9950 10100 3    50   ~ 10
 OUT_7
@@
 Wire Wire Line
 	10550 10100 10550 10400
-Text Label 4550 6450 0    50   ~ 10
-CRNK_MCU
 Text Label 8000 11400 0    50   ~ 10
 5V1
@@
 Text Label 8900 11450 0    50   ~ 0
 V5V
-Text Label 4050 6250 2    50   ~ 10
+Text Label 4050 6050 2    50   ~ 10
 5V1
-Text Label 4550 6250 0    50   ~ 10
+Text Label 4550 6050 0    50   ~ 10
 5V2
 Text Label 8750 6700 1    50   ~ 10
@@
 Text Label 9250 6700 1    50   ~ 10
 DFB_8
-Text Label 4050 5050 2    50   ~ 10
+Text Label 4050 4950 2    50   ~ 10
 OUT_10
-Text Label 4050 4950 2    50   ~ 10
+Text Label 4050 4850 2    50   ~ 10
 DFB_10
+Text Label 4550 4850 0    50   ~ 10
+OUT_9
 Text Label 4550 4950 0    50   ~ 10
-OUT_9
-Text Label 4550 5050 0    50   ~ 10
 OUT_8
-Text Label 4050 4850 2    50   ~ 10
+Text Label 4050 4750 2    50   ~ 10
 DFB_9
-Text Label 4550 4850 0    50   ~ 10
+Text Label 4550 4750 0    50   ~ 10
 DFB_8
 Text Label 8100 7300 2    50   ~ 10
@@
 Text Label 8000 8200 2    50   ~ 10
 OUT_24
+Text Label 4050 5150 2    50   ~ 10
+OUT_11
 Text Label 4050 5250 2    50   ~ 10
-OUT_11
+OUT_12
 Text Label 4050 5350 2    50   ~ 10
-OUT_12
-Text Label 4050 5450 2    50   ~ 10
 OUT_13
-Text Label 4050 5150 2    50   ~ 10
+Text Label 4050 5050 2    50   ~ 10
 DFB_11
-Text Label 4550 5450 0    50   ~ 10
+Text Label 4550 5350 0    50   ~ 10
 DFB_12
-Text Label 4550 5350 0    50   ~ 10
+Text Label 4550 5250 0    50   ~ 10
 DFB_13
-Text Label 4550 5150 0    50   ~ 10
+Text Label 4550 5050 0    50   ~ 10
 OUT_5
-Text Label 4550 5750 0    50   ~ 10
-OUT_24
 Text Label 8000 8400 2    50   ~ 10
 OUT_23
@@
 Text Label 8000 8900 2    50   ~ 10
 OUT_6
-Text Label 4050 5650 2    50   ~ 10
+Text Label 4550 5450 0    50   ~ 10
 OUT_23
-Text Label 4050 5750 2    50   ~ 10
-OUT_21
 Text Label 7350 9200 2    50   ~ 10
 IGN_OUT_1
@@
 Text Label 8100 9500 2    50   ~ 10
 IGN_OUT_4
-Text Label 4050 5950 2    50   ~ 10
-IGN_OUT_3
-Text Label 4550 5950 0    50   ~ 10
-IGN_OUT_4
-Text Label 4050 5850 2    50   ~ 10
-IGN_OUT_1
 Text Label 10250 10450 0    50   ~ 10
 OUT_19
 Text Label 10150 10550 0    50   ~ 10
 OUT_20
-Text Label 4050 6450 2    50   ~ 10
-OUT_19
 Text Label 12550 5550 0    50   ~ 10
 12V
@@
 Text Label 15050 7950 0    50   ~ 10
 CAN_H
-Text Label 4550 5550 0    60   ~ 12
+Text Label 4550 6550 0    60   ~ 12
 V5V
 $Comp
@@
 Text Label 4050 3450 2    60   ~ 12
 GND
-Text Label 4050 3650 2    50   ~ 10
+Text Label 4050 6450 2    50   ~ 10
 12V
 Text Label 8100 7800 2    50   ~ 0
 LIN_IO
-Text Label 5950 6350 2    50   ~ 0
-LIN_IO
-Text Label 4550 5250 0    50   ~ 10
+Text Label 4550 5150 0    50   ~ 10
 OUT_6
-Text Label 4550 5850 0    50   ~ 10
-IGN_OUT_2
-Text Label 4550 5650 0    50   ~ 10
+Text Label 4550 5550 0    50   ~ 10
 OUT_22
 Text Label 10750 10100 3    50   ~ 0
@@
 Text Label 10650 10100 3    50   ~ 0
 LIN_TX
-Text Label 6000 6250 2    50   ~ 0
-LIN_RX
-Text Label 5750 6150 0    50   ~ 0
+Text Label 2900 3200 0    50   ~ 0
 LIN_TX
+Text Label 4050 3750 2    50   ~ 10
+INJ_IN_2
 Text Label 4050 3850 2    50   ~ 10
-INJ_IN_2
+INJ_IN_4
+Text Label 2400 3000 2    50   ~ 10
+CAN_L
 Text Label 4050 3950 2    50   ~ 10
-INJ_IN_4
-Text Label 2750 4100 2    50   ~ 10
-CAN_L
+IGN_IN_2
 Text Label 4050 4050 2    50   ~ 10
-IGN_IN_2
+IGN_IN_4
 Text Label 4050 4150 2    50   ~ 10
-IGN_IN_4
+IN_10
 Text Label 4050 4250 2    50   ~ 10
-IN_10
-Text Label 4050 4350 2    50   ~ 10
 IN_12
-Text Label 2750 4000 2    50   ~ 10
+Text Label 2900 3000 0    50   ~ 10
 CAN_TX
+Text Label 4550 3750 0    50   ~ 10
+INJ_IN_3
+Text Label 4050 3650 2    60   ~ 12
+VDD
+Text Label 2400 3100 2    50   ~ 10
+CAN_H
+Text Label 4550 3650 0    50   ~ 10
+INJ_IN_1
 Text Label 4550 3850 0    50   ~ 10
-INJ_IN_3
-Text Label 4050 3750 2    60   ~ 12
-VDD
-Text Label 3000 4100 0    50   ~ 10
-CAN_H
-Text Label 4550 3750 0    50   ~ 10
-INJ_IN_1
+IGN_IN_1
 Text Label 4550 3950 0    50   ~ 10
-IGN_IN_1
+IGN_IN_3
 Text Label 4550 4050 0    50   ~ 10
-IGN_IN_3
+IN_9
 Text Label 4550 4150 0    50   ~ 10
-IN_9
-Text Label 4550 4250 0    50   ~ 10
 IN_11
-Text Label 3000 4000 0    50   ~ 10
+Text Label 2900 2900 0    50   ~ 10
 CAN_RX
 Wire Wire Line
@@
 Wire Wire Line
 	12850 6550 12850 6750
-Text Label 4050 6550 2    50   ~ 10
+Text Label 4050 6350 2    50   ~ 10
 CRNK+
-Text Label 4550 6550 0    50   ~ 10
-CRNK-
-Text Label 4550 6350 0    50   ~ 10
-OUT_20
-Text Label 4050 6350 2    50   ~ 10
-OUT_7
-Text Label 4050 5550 2    60   ~ 12
+Text Label 4050 6550 2    60   ~ 12
 V5V
 Text Label 4050 6650 2    60   ~ 12
@@
 Text Label 4550 3550 0    60   ~ 12
 V5V
+Text Label 4550 6350 0    50   ~ 10
+CRNK-
+Text Label 4550 5650 0    50   ~ 10
+IGN_OUT_2
+Text Label 4550 5750 0    50   ~ 10
+IGN_OUT_4
+Text Label 4050 5450 2    50   ~ 10
+OUT_24
+Text Label 4550 6250 0    50   ~ 10
+CRNK_MCU
+Text Label 4550 5850 0    50   ~ 10
+SDO
+Text Label 4550 5950 0    50   ~ 10
+FCLP
+Text Label 4050 6250 2    50   ~ 10
+OUT_19
+Text Label 4050 5650 2    50   ~ 10
+IGN_OUT_1
+Text Label 4050 5750 2    50   ~ 10
+IGN_OUT_3
+Text Label 4050 5550 2    50   ~ 10
+OUT_21
+Text Label 4050 5850 2    50   ~ 10
+CSN
+Text Label 4050 6150 2    50   ~ 10
+OUT_7
+Text Label 4550 6150 0    50   ~ 10
+OUT_20
+$Comp
+L Mechanical:Heatsink HS1
+U 1 1 5CDB3DEE
+P 7100 4850
+F 0 "HS1" H 7242 4971 50  0000 L CNN
+F 1 "Heatsink" H 7242 4880 50  0000 L CNN
+F 2 "Heatsink:HEATSINK" H 7112 4850 50  0001 C CNN
+F 3 "~" H 7112 4850 50  0001 C CNN
+	1    7100 4850
+	1    0    0    -1
+$EndComp
+$Comp
+L Connector_Generic:Conn_02x04_Odd_Even J3
+U 1 1 5CE5CF8D
+P 2600 3000
+F 0 "J3" H 2650 3317 50  0000 C CNN
+F 1 "Conn_02x04_Odd_Even" H 2650 3226 50  0000 C CNN
+F 2 "Connector_PinHeader_1.00mm:PinHeader_2x04_P1.00mm_Vertical" H 2600 3000 50  0001 C CNN
+F 3 "~" H 2600 3000 50  0001 C CNN
+	1    2600 3000
+	1    0    0    -1
+$EndComp
+Text Label 2400 3200 2    50   ~ 0
+LIN_IO
+Text Label 2900 3100 0    50   ~ 0
+LIN_RX
+$Comp
+L Mechanical:Heatsink HS2
+U 1 1 5CF47684
+P 7100 5350
+F 0 "HS2" H 7242 5471 50  0000 L CNN
+F 1 "Heatsink" H 7242 5380 50  0000 L CNN
+F 2 "Heatsink:HEATSINK" H 7112 5350 50  0001 C CNN
+F 3 "~" H 7112 5350 50  0001 C CNN
+	1    7100 5350
+	1    0    0    -1
+$EndComp
 $EndSCHEMATC
