File: TLE8888_Module/TLE8888_Module.sch (KiCad schematic (older format))
At the start: 44 parts, among them J1 Conn_01x01, J2 Conn_02x39_Odd_Even, J3 Conn_02x04_Odd_Even, Q1 IPD30N06S2L-23, U2 TLE8888QK

Commit message: sync
Parts:
- added D10, D11, D13, D14, D15, D16, D17, D3, D4, D5, D7, D8, D9: LED, LED_SMD:LED_0603_1608Metric_Pad1.05x0.95mm_HandSolder, symbol Device:LED
- added R1, R11, R14, R24, R25, R26, R27, R28, R30, R31, R32, R33, R34: 1K, Resistor_SMD:R_0603_1608Metric_Pad1.05x0.95mm_HandSolder, symbol Device:R
- added R23: TLE8888 LOGO, Symbol:TLE8888, symbol Device:R
- C1, C10, C11, C12, C13, C14, C15, C16, C3, C4, C5, C6, C7, C8, C9: footprint Capacitor_SMD:C_0805_2012Metric_Pad1.15x1.40mm_HandSolder -> Capacitor_SMD:C_0603_1608Metric_Pad1.05x0.95mm_HandSolder
- J3: footprint Connector_PinHeader_1.00mm:PinHeader_2x04_P1.00mm_Vertical -> Connector_PinHeader_2.54mm:PinHeader_2x04_P2.54mm_Vertical
- R10, R12, R13, R15, R16, R17, R18, R19, R2, R20, R21, R22, R3, R4, R5, R6, R7, R8, R9: footprint Resistor_SMD:R_0805_2012Metric_Pad1.15x1.40mm_HandSolder -> Resistor_SMD:R_0603_1608Metric_Pad1.05x0.95mm_HandSolder
Connections:
- wire segments 153 -> 167
Other:
- moved on the sheet: J1

Commit message: cleaned up
Parts:
- C1, C10, C13, C4, C5, C6: value 100nF 50V -> 100nF; Manufacturer WURTH -> (none); Part # 885012208087 -> (none); VEND MOUSER -> (none); VEND# 710-885012208087 -> (none)
- C11: value 4.7nF 50V -> 4.7nF; Manufacturer WURTH -> (none); Part # 885012208079 -> (none); VEND# 710-885012208079 -> (none)
- C12, C15: value C -> 1nF; Manufacturer WURTH -> (none); Part # 885012208087 -> (none); VEND MOUSER -> (none); VEND# 710-885012208087 -> (none)
- C14, C16: value 100nF 100V -> 100nF; Manufacturer WURTH -> (none); Part # 885012208087 -> (none); VEND MOUSER -> (none); VEND# 710-885012208087 -> (none)
- C2: Manufacturer NICHICON -> (none)
- C3: Manufacturer WURTH -> (none); Part # 885012208050 -> (none); VEND# 710-885012208050 -> (none)
- C7: value 10uF 50V -> 10uF; Manufacturer MURATA -> (none); Part # GRT31CR61H106KE01L -> (none); VEND MOUSER -> (none); VEND# 81-GRT31CR61H106KE1L -> (none)
- C8, C9: value 10uF 25V -> 10uF; Manufacturer MURATA -> (none); Part # GRT31CR61H106KE01L -> (none); VEND MOUSER -> (none); VEND# 81-GRT31CR61H106KE1L -> (none)
- D1: Manufacturer ON-SEMI -> (none)
- D2: symbol BOSCH_154_PIN:PESD1CAN-UX -> Power_Protection:SP0502BAHT; Manufacturer Nexperia USA Inc. -> (none)
- Q1: Manufacturer INFINEON -> (none)
- R22: value 120 -> 120R
- R23: value TLE8888 LOGO -> TLE8888 LOGO DNP; VEND MOUSER -> (none)
- U2: symbol BOSCH_154_PIN:TLE8888QK -> TLE8888:TLE8888QK; Manufacturer INFINEON -> (none)
Connections:
- wire segments 167 -> 166
