File: TLE8888_Module/TLE8888_Module.sch (KiCad schematic (older format))
At the start: 71 parts, among them J1 Conn_01x01, J2 Conn_02x39_Odd_Even, J3 Conn_02x04_Odd_Even, Q1 IPD30N06S2L-23, U2 TLE8888QK

Commit message: manual sync with 960
Parts:
- D2: symbol BOSCH_154_PIN:PESD1CAN-UX -> Power_Protection:SP0502BAHT
- U2: symbol BOSCH_154_PIN:TLE8888QK -> TLE8888:TLE8888QK
Connections:
- wire segments 167 -> 166
Changed lines of the file:
@@
 $EndDescr
 $Comp
-L BOSCH_154_PIN:TLE8888QK U2
+L TLE8888:TLE8888QK U2
 U 1 1 5C5DF903
 P 10150 6950
@@
 	14325 7250 14325 7500
 $Comp
-L BOSCH_154_PIN:PESD1CAN-UX D2
+L Power_Protection:SP0502BAHT D2
 U 1 1 5C984DE7
-P 14825 7600
+P 14525 7600
 AR Path="/5C984DE7" Ref="D2"  Part="1"
 AR Path="/5C5D7FA6/5C984DE7" Ref="D2"  Part="1"
-F 0 "D2" H 15125 7750 60  0000 C CNN
-F 1 "PESD1CAN-UX" H 15375 7475 60  0000 C CNN
-F 2 "Package_TO_SOT_SMD:SOT-323_SC-70_Handsoldering" H 15025 7800 60  0001 L CNN
-F 3 "https://assets.nexperia.com/documents/data-sheet/PESD1CAN-U.pdf" H 15025 7900 60  0001 L CNN
-F 4 "Active" H 15025 8800 60  0001 L CNN "Status"
-F 5 "MOUSER" H 75  -700 50  0001 C CNN "VEND"
-F 6 "PESD1CANUX" H 75  -700 50  0001 C CNN "Part #"
-F 7 "771-PESD1CANUX" H 75  -700 50  0001 C CNN "VEND#"
-	1    14825 7600
-	1    0    0    -1
+F 0 "D2" H 14825 7750 60  0000 C CNN
+F 1 "PESD1CAN-UX" H 15075 7475 60  0000 C CNN
+F 2 "Package_TO_SOT_SMD:SOT-323_SC-70_Handsoldering" H 14725 7800 60  0001 L CNN
+F 3 "https://assets.nexperia.com/documents/data-sheet/PESD1CAN-U.pdf" H 14725 7900 60  0001 L CNN
+F 4 "Active" H 14725 8800 60  0001 L CNN "Status"
+F 5 "MOUSER" H -225 -700 50  0001 C CNN "VEND"
+F 6 "PESD1CANUX" H -225 -700 50  0001 C CNN "Part #"
+F 7 "771-PESD1CANUX" H -225 -700 50  0001 C CNN "VEND#"
+	1    14525 7600
+	0    -1   -1   0
 $EndComp
 $Comp
 L power:GND #PWR022
 U 1 1 5C99C043
-P 15125 7600
-F 0 "#PWR022" H 15125 7350 50  0001 C CNN
-F 1 "GND" H 15130 7427 50  0000 C CNN
-F 2 "" H 15125 7600 50  0001 C CNN
-F 3 "" H 15125 7600 50  0001 C CNN
-	1    15125 7600
+P 14725 7600
+F 0 "#PWR022" H 14725 7350 50  0001 C CNN
+F 1 "GND" H 14730 7427 50  0000 C CNN
+F 2 "" H 14725 7600 50  0001 C CNN
+F 3 "" H 14725 7600 50  0001 C CNN
+	1    14725 7600
 	0    -1   -1   0
 $EndComp
-Wire Wire Line
-	15125 7600 15140 7600
 $Comp
 L power:GND #PWR06
