File: TLE8888_Module/TLE8888_Module.sch (KiCad schematic (older format))
At the start: 71 parts, among them J1 Conn_01x01, J2 Conn_02x39_Odd_Even, J3 Conn_02x04_Odd_Even, Q1 IPD30N06S2L-23, U2 TLE8888QK

Commit message: V 0.2
Parts:
- removed HS1, HS2: Heatsink, Heatsink:HEATSINK, symbol Mechanical:Heatsink
- C12, C15: value 1nF -> DNP
- J1: value Conn_01x01 -> DNP CORNER HOLE
- R12, R13, R15, R16, R17, R18, R19, R9: value 0 -> DNP
Connections:
- wire segments 166 -> 164
Other:
- moved on the sheet: D11, D17, D5, D8, J1, R14, R9
