File: TLE8888_Module/TLE8888_Module.kicad_pcb (KiCad board)
At the start: 4 copper layers, 100 x 22 mm, 41 parts, among them J1 Conn_01x01, J2 Conn_02x39_Odd_Even, Q1 IPD30N06S2L-23, U2 TLE8888QK

Commit message: sync
Parts:
- added HS1: Heatsink, Heatsink:HEATSINK, F.Cu at (95.4, 25.9)
- added HS2: Heatsink, Heatsink:HEATSINK, B.Cu at (68.8, 32.5)
- added J3: Conn_02x04_Odd_Even, Connector_PinHeader_1.00mm:PinHeader_2x04_P1.00mm_Vertical, F.Cu at (40.5, 31.2)
- C2: moved to F.Cu
- moved C2 79.3 mm to (113.0, 27.1)
- moved R21 69.6 mm to (117.3, 27.7), turned to 180 degrees
- moved C16 67.9 mm to (117.2, 23.4), turned to 0 degrees
- moved C1 65.7 mm to (117.3, 25.5), turned to 0 degrees
- moved D1 60.0 mm to (102.0, 26.3)
- moved C5 22.5 mm to (88.3, 31.5), turned to 270 degrees
- moved C4 22.0 mm to (85.2, 30.2), turned to 90 degrees
- moved C11 15.3 mm to (81.0, 26.0)
- moved R16 11.2 mm to (105.7, 34.3), turned to 90 degrees
- moved R15 11.0 mm to (100.8, 32.3), turned to 90 degrees
- moved C15 11.0 mm to (102.9, 32.3), turned to 90 degrees
- moved R17 10.9 mm to (107.8, 34.3), turned to 90 degrees
- moved C10 10.8 mm to (81.0, 22.2), turned to 90 degrees
- moved C8 10.8 mm to (85.1, 22.2), turned to 90 degrees
- moved C9 10.8 mm to (83.1, 22.2), turned to 90 degrees
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Connections:
- J2 pad 10: /INJ_IN_3 -> /IGN_IN_1
- J2 pad 11: /INJ_IN_4 -> /IGN_IN_2
- J2 pad 12: /IGN_IN_1 -> /IGN_IN_3
- J2 pad 13: /IGN_IN_2 -> /IGN_IN_4
- J2 pad 14: /IGN_IN_3 -> /IN_9
- J2 pad 15: /IGN_IN_4 -> /IN_10
- J2 pad 16: /IN_9 -> /IN_11
- J2 pad 17: /IN_10 -> /IN_12
- J2 pad 18: /IN_11 -> /OUT_18
- J2 pad 19: /IN_12 -> /OUT_16
- J2 pad 20: /CAN_RX -> /OUT_17
- J2 pad 21: /CAN_TX -> /OUT_2
- J2 pad 22: /CAN_H -> /OUT_1
- J2 pad 23: /CAN_L -> /OUT_4
- J2 pad 24: /OUT_18 -> /OUT_3
- J2 pad 25: /OUT_16 -> /OUT_15
- J2 pad 26: /OUT_17 -> /OUT_14
- J2 pad 27: /OUT_2 -> /DFB_9
- J2 pad 28: /OUT_1 -> /DFB_8
- J2 pad 29: /OUT_4 -> /DFB_10
- J2 pad 30: /OUT_3 -> /OUT_9
- J2 pad 31: /OUT_15 -> /OUT_10
- J2 pad 32: /OUT_14 -> /OUT_8
- J2 pad 33: /DFB_9 -> /DFB_11
- J2 pad 34: /DFB_8 -> /OUT_5
- J2 pad 35: /DFB_10 -> /OUT_11
- J2 pad 36: /OUT_9 -> /OUT_6
- J2 pad 37: /OUT_10 -> /OUT_12
- J2 pad 38: /OUT_8 -> /DFB_13
- J2 pad 39: /DFB_11 -> /OUT_13
- J2 pad 40: /OUT_5 -> /DFB_12
- J2 pad 41: /OUT_11 -> /OUT_24
- J2 pad 42: /OUT_6 -> /OUT_23
- J2 pad 43: /OUT_12 -> /OUT_21
- J2 pad 44: /DFB_13 -> /OUT_22
- J2 pad 45: /OUT_13 -> /IGN_OUT_1
- J2 pad 46: /DFB_12 -> /IGN_OUT_2
- J2 pad 47: /OUT_23 -> /IGN_OUT_3
- J2 pad 48: /OUT_22 -> /IGN_OUT_4
- J2 pad 49: /OUT_21 -> /CSN
- J2 pad 5: /12V -> /VDD
- J2 pad 50: /OUT_24 -> /SDO
- J2 pad 51: /IGN_OUT_1 -> /SIP
- J2 pad 52: /IGN_OUT_2 -> /FCLP
- J2 pad 53: /IGN_OUT_3 -> /5V1
- J2 pad 54: /IGN_OUT_4 -> /5V2
- J2 pad 55: /CSN -> /OUT_7
- J2 pad 56: /SDO -> /OUT_20
- J2 pad 57: /SIP -> /OUT_19
- J2 pad 58: /FCLP -> /CRNK_MCU
- J2 pad 59: /5V1 -> /CRNK+
- J2 pad 6: /12V -> /INJ_IN_1
- J2 pad 60: /5V2 -> /CRNK-
- J2 pad 61: /OUT_7 -> /12V
- J2 pad 62: /OUT_20 -> /12V
- J2 pad 63: /OUT_19 -> /V5V
- J2 pad 64: /CRNK_MCU -> /V5V
- J2 pad 65: /CRNK+ -> GND
- J2 pad 66: /CRNK- -> GND
- J2 pad 7: /VDD -> /INJ_IN_2
- J2 pad 8: /INJ_IN_1 -> /INJ_IN_3
- J2 pad 9: /INJ_IN_2 -> /INJ_IN_4
Routing:
- net Net-(D1-Pad1): track 69.6 -> 7.49 mm
- net /LIN_IO: track 0.00 -> 36.1 mm, vias 0 -> 2
- net /LIN_TX: track 0.00 -> 35.3 mm, vias 0 -> 1
- net /LIN_RX: track 0.00 -> 35.1 mm, vias 0 -> 1
- net /MAIN_RELAY: track 0.00 -> 22.4 mm
- net /CAN_TX: track 39.3 -> 23.0 mm
- net /VDD: track 94.6 -> 78.6 mm, vias 2 -> 0
- net /12V: track 81.8 -> 94.6 mm, vias 3 -> 5
- net /CAN_RX: track 36.8 -> 24.1 mm
- net Net-(C12-Pad1): track 56.5 -> 49.3 mm
- net /CAN_H: track 34.6 -> 27.4 mm
- net /KEY: track 11.2 -> 4.43 mm
- net /INJ_IN_2: track 56.0 -> 49.3 mm
- net /INJ_IN_1: track 54.2 -> 47.6 mm
- net /CRNK+: track 24.2 -> 17.8 mm
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
Commit message: sync
Parts:
- removed HS1, HS2: Heatsink, Heatsink:HEATSINK
- added D10: LED, LED_SMD:LED_0603_1608Metric_Pad1.05x0.95mm_HandSolder, F.Cu at (46.5, 25.5)
- added D11: LED, LED_SMD:LED_0603_1608Metric_Pad1.05x0.95mm_HandSolder, F.Cu at (39.9, 25.5)
- added D13: LED, LED_SMD:LED_0603_1608Metric_Pad1.05x0.95mm_HandSolder, F.Cu at (43.2, 25.5)
- added D14: LED, LED_SMD:LED_0603_1608Metric_Pad1.05x0.95mm_HandSolder, F.Cu at (48.1, 25.5)
- added D15: LED, LED_SMD:LED_0603_1608Metric_Pad1.05x0.95mm_HandSolder, F.Cu at (33.3, 25.5)
- added D16: LED, LED_SMD:LED_0603_1608Metric_Pad1.05x0.95mm_HandSolder, F.Cu at (31.6, 25.5)
- added D17: LED, LED_SMD:LED_0603_1608Metric_Pad1.05x0.95mm_HandSolder, F.Cu at (105.9, 32.9)
- added D3: LED, LED_SMD:LED_0603_1608Metric_Pad1.05x0.95mm_HandSolder, F.Cu at (34.9, 25.6)
- added D4: LED, LED_SMD:LED_0603_1608Metric_Pad1.05x0.95mm_HandSolder, F.Cu at (44.8, 25.5)
- added D5: LED, LED_SMD:LED_0603_1608Metric_Pad1.05x0.95mm_HandSolder, F.Cu at (41.5, 25.5)
- added D7: LED, LED_SMD:LED_0603_1608Metric_Pad1.05x0.95mm_HandSolder, F.Cu at (38.2, 25.5)
- added D8: LED, LED_SMD:LED_0603_1608Metric_Pad1.05x0.95mm_HandSolder, F.Cu at (36.6, 25.5)
- added D9: LED, LED_SMD:LED_0603_1608Metric_Pad1.05x0.95mm_HandSolder, F.Cu at (49.8, 25.5)
- added R1: 1K, Resistor_SMD:R_0603_1608Metric_Pad1.05x0.95mm_HandSolder, B.Cu at (35.0, 25.6)
- added R11: 1K, Resistor_SMD:R_0603_1608Metric_Pad1.05x0.95mm_HandSolder, B.Cu at (44.8, 25.5)
- added R14: 1K, Resistor_SMD:R_0603_1608Metric_Pad1.05x0.95mm_HandSolder, B.Cu at (41.5, 25.5)
- added R23: 1K, Symbol:TLE8888, B.Cu at (43.3, 20.1)
- added R23: 1K, Symbol:TLE8888, F.Cu at (41.7, 20.8)
- added R24: 1K, Resistor_SMD:R_0603_1608Metric_Pad1.05x0.95mm_HandSolder, B.Cu at (38.2, 25.5)
- added R25: 1K, Resistor_SMD:R_0603_1608Metric_Pad1.05x0.95mm_HandSolder, B.Cu at (36.6, 25.5)
- added R26: 1K, Resistor_SMD:R_0603_1608Metric_Pad1.05x0.95mm_HandSolder, B.Cu at (49.8, 25.5)
- added R27: 1K, Resistor_SMD:R_0603_1608Metric_Pad1.05x0.95mm_HandSolder, B.Cu at (46.5, 25.5)
- added R28: 1K, Resistor_SMD:R_0603_1608Metric_Pad1.05x0.95mm_HandSolder, B.Cu at (39.9, 25.5)
- added R30: 1K, Resistor_SMD:R_0603_1608Metric_Pad1.05x0.95mm_HandSolder, B.Cu at (43.2, 25.5)
- added R31: 1K, Resistor_SMD:R_0603_1608Metric_Pad1.05x0.95mm_HandSolder, B.Cu at (48.1, 25.5)
- added R32: 1K, Resistor_SMD:R_0603_1608Metric_Pad1.05x0.95mm_HandSolder, B.Cu at (33.3, 25.5)
- added R33: 1K, Resistor_SMD:R_0603_1608Metric_Pad1.05x0.95mm_HandSolder, B.Cu at (31.6, 25.5)
- added R34: 1K, Resistor_SMD:R_0603_1608Metric_Pad1.05x0.95mm_HandSolder, F.Cu at (105.3, 29.0)
- C1, C10, C11, C12, C15, C16, C4, C5, C6, C7, C8, C9: footprint Capacitor_SMD:C_0805_2012Metric_Pad1.15x1.40mm_HandSolder -> Capacitor_SMD:C_0603_1608Metric_Pad1.05x0.95mm_HandSolder
- C13, C14, C3: footprint Capacitor_SMD:C_0805_2012Metric_Pad1.15x1.40mm_HandSolder -> Capacitor_SMD:C_0603_1608Metric_Pad1.05x0.95mm_HandSolder; moved to F.Cu
- J3: footprint Connector_PinHeader_1.00mm:PinHeader_2x04_P1.00mm_Vertical -> Connector_PinHeader_2.54mm:PinHeader_2x04_P2.54mm_Vertical
- R10, R2, R20, R3, R4, R5, R6, R7, R8: footprint Resistor_SMD:R_0805_2012Metric_Pad1.15x1.40mm_HandSolder -> Resistor_SMD:R_0603_1608Metric_Pad1.05x0.95mm_HandSolder; moved to F.Cu
- R12, R13, R15, R16, R17, R18, R19, R21, R22, R9: footprint Resistor_SMD:R_0805_2012Metric_Pad1.15x1.40mm_HandSolder -> Resistor_SMD:R_0603_1608Metric_Pad1.05x0.95mm_HandSolder
- moved C7 94.4 mm to (117.3, 31.6), turned to 0 degrees
- moved C6 94.4 mm to (117.3, 33.3), turned to 0 degrees
- moved R10 26.1 mm to (85.5, 22.4), turned to 90 degrees
- moved R8 24.7 mm to (83.9, 22.4), turned to 90 degrees
- moved J3 16.5 mm to (24.1, 33.5), turned to 180 degrees
- moved R22 10.1 mm to (56.3, 26.2), turned to 270 degrees
- moved D2 8.77 mm to (53.1, 25.1), turned to 180 degrees
- moved R7 6.66 mm to (82.4, 22.4), turned to 90 degrees
- moved R2 6.56 mm to (81.5, 32.1)
- moved C11 5.50 mm to (86.5, 26.7), turned to 90 degrees
- moved R16 4.22 mm to (106.2, 30.1), turned to 270 degrees
- moved R17 4.19 mm to (107.8, 30.1), turned to 270 degrees
- moved R4 3.99 mm to (81.5, 30.6)
- moved C13 3.78 mm to (59.0, 24.6)
- moved R19 3.22 mm to (106.2, 33.5), turned to 90 degrees
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Connections:
- J2 pad 59: /CRNK+ -> /CRNK-
- J2 pad 60: /CRNK- -> /CRNK+
- J3 pad 2: /CAN_RX -> /CAN_H
- J3 pad 4: /CAN_TX -> /LIN_IO
- J3 pad 5: /CAN_H -> /CAN_TX
- J3 pad 6: /LIN_RX -> /CAN_RX
- J3 pad 7: /LIN_IO -> /LIN_TX
- J3 pad 8: /LIN_TX -> /LIN_RX
Routing:
- net /IGN_OUT_1: track 19.7 -> 69.0 mm, vias 0 -> 2
- net /OUT_21: track 18.6 -> 63.8 mm, vias 1 -> 2
- net /V5V: track 19.9 -> 62.8 mm, vias 6 -> 9
- net /OUT_5: track 7.01 -> 45.8 mm, vias 0 -> 2
- net /MAIN_RELAY: track 22.4 -> 57.4 mm, vias 0 -> 1
- net /12V: track 94.6 -> 128.0 mm, vias 5 -> 7
- net /LIN_IO: track 36.1 -> 67.8 mm, vias 2 -> 1
- net /CAN_H: track 27.4 -> 58.3 mm, vias 0 -> 1
- net /OUT_18: track 20.2 -> 50.7 mm, vias 0 -> 2
- net /IGN_IN_1: track 42.6 -> 70.7 mm, vias 0 -> 2
- net /CAN_L: track 28.4 -> 53.6 mm, vias 0 -> 1
- net /INJ_IN_1: track 47.6 -> 72.7 mm, vias 0 -> 2
- net /CAN_RX: track 24.1 -> 48.4 mm, vias 0 -> 1
- net /VDD: track 78.6 -> 102.6 mm, vias 0 -> 5
- net /OUT_8: track 7.77 -> 31.5 mm, vias 0 -> 1
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Other:
- board text added: "12V"
- board text added: "5V"
- board text added: "5V1"
- board text added: "5V2"
- board text added: "BFB10"
- board text added: "CAN_H"
- board text added: "CAN_L"
- board text added: "CAN_RX"
- board text added: "CAN_TX"
- board text added: "CRANK OUT"
- board text added: "CRNK+"
- board text added: "CRNK-"
- board text added: "CRNK_IN"
- board text added: "CSN"
- board text added: "DFB11"
- board text added: "DFB12"
- board text added: "DFB13"
- board text added: "DFB8"
- board text added: "DFB9"
- board text added: "FCLP"
- board text added: "GND"
- board text added: "IGN1"
- board text added: "IGN2"
- board text added: "IGN3"
- board text added: "IGN4"
- board text added: "IN1"
- board text added: "IN10"
- board text added: "IN11"
- board text added: "IN12"
- board text added: "IN2"
- board text added: "IN3"
- board text added: "IN9"
- board text added: "I_IN1"
- board text added: "I_IN2"
- board text added: "I_IN3"
- board text added: "I_IN4"
- board text added: "LIN_IO"
- board text added: "LIN_RX"
- board text added: "LIN_TX"
- board text added: "MAIN_RLY"
- board text added: "OUT1"
- board text added: "OUT10"
- board text added: "OUT11"
- board text added: "OUT12"
- board text added: "OUT13"
- board text added: "OUT14"
- board text added: "OUT15"
- board text added: "OUT16"
- board text added: "OUT17"
- board text added: "OUT18"
- board text added: "OUT19"
- board text added: "OUT2"
- board text added: "OUT20"
- board text added: "OUT21"
- board text added: "OUT22"
- board text added: "OUT23"
- board text added: "OUT24"
- board text added: "OUT3"
- board text added: "OUT4"
- board text added: "OUT5"
- board text added: "OUT6"
- board text added: "OUT7"
- board text added: "OUT8"
- board text added: "OUT9"
- board text added: "SDO"
- board text added: "SIP"
- board text added: "VDD"
- board text removed: "TLE8888-QK"

Commit message: sync
Routing:
- net /5V2: track 40.5 -> 42.6 mm

Commit message: manual sync with 960
Parts:
- C1, C10, C13, C4, C5, C6: value 100nF 50V -> 100nF
- C11: value 4.7nF 50V -> 4.7nF
- C12, C15: value C -> 1nF
- C14, C16: value 100nF 100V -> 100nF
- C7: value 10uF 50V -> 10uF
- C8, C9: value 10uF 25V -> 10uF
- R22: value 120 -> 120R
- R23 (x2): value 1K -> TLE8888 LOGO DNP
Connections:
- D2 pad 1: /CAN_L -> /CAN_H
- D2 pad 2: /CAN_H -> /CAN_L
Changed lines of the file:
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@@
   )
   (setup
-    (last_trace_width 0.3048)
+    (last_trace_width 0.1524)
     (user_trace_width 0.1524)
     (user_trace_width 0.2159)
@@
       (effects (font (size 1 1) (thickness 0.15)) (justify mirror))
     )
-    (fp_text value 1K (at 0 0.5 180) (layer B.Fab)
+    (fp_text value "TLE8888 LOGO DNP" (at 0 0.5 180) (layer B.Fab)
       (effects (font (size 1 1) (thickness 0.15)) (justify mirror))
     )
@@
       (effects (font (size 1 1) (thickness 0.15)))
     )
-    (fp_text value 1K (at 0 -0.5) (layer F.Fab)
+    (fp_text value "TLE8888 LOGO DNP" (at 0 -0.5) (layer F.Fab)
       (effects (font (size 1 1) (thickness 0.15)))
     )
@@
       (effects (font (size 0.5 0.5) (thickness 0.1)))
     )
-    (fp_text value 120 (at 0 1.43 270) (layer F.Fab)
+    (fp_text value 120R (at 0 1.43 270) (layer F.Fab)
       (effects (font (size 1 1) (thickness 0.15)))
     )
@@
       (effects (font (size 0.5 0.5) (thickness 0.1)) (justify mirror))
     )
-    (fp_text value "100nF 100V" (at 0 -1.43) (layer B.Fab)
+    (fp_text value 100nF (at 0 -1.43) (layer B.Fab)
       (effects (font (size 1 1) (thickness 0.15)) (justify mirror))
     )
@@
       (effects (font (size 0.5 0.5) (thickness 0.1)) (justify mirror))
     )
-    (fp_text value C (at 0 -1.43 270) (layer B.Fab)
+    (fp_text value 1nF (at 0 -1.43 270) (layer B.Fab)
       (effects (font (size 1 1) (thickness 0.15)) (justify mirror))
     )
@@
       (effects (font (size 0.5 0.5) (thickness 0.1)))
     )
-    (fp_text value "100nF 100V" (at 0 1.43) (layer F.Fab)
+    (fp_text value 100nF (at 0 1.43) (layer F.Fab)
       (effects (font (size 1 1) (thickness 0.15)))
     )
@@
       (effects (font (size 0.5 0.5) (thickness 0.1)))
     )
-    (fp_text value "100nF 50V" (at 0 1.43 180) (layer F.Fab)
+    (fp_text value 100nF (at 0 1.43 180) (layer F.Fab)
       (effects (font (size 1 1) (thickness 0.15)))
     )
@@
       (effects (font (size 0.5 0.5) (thickness 0.1)) (justify mirror))
     )
-    (fp_text value C (at 0 -1.43 270) (layer B.Fab)
+    (fp_text value 1nF (at 0 -1.43 270) (layer B.Fab)
       (effects (font (size 1 1) (thickness 0.15)) (justify mirror))
     )
@@
       (effects (font (size 0.5 0.5) (thickness 0.1)) (justify mirror))
     )
-    (fp_text value "4.7nF 50V" (at 0 -1.43 90) (layer B.Fab)
+    (fp_text value 4.7nF (at 0 -1.43 90) (layer B.Fab)
       (effects (font (size 1 1) (thickness 0.15)) (justify mirror))
     )
@@
       (effects (font (size 0.5 0.5) (thickness 0.1)) (justify mirror))
     )
-    (fp_text value "100nF 50V" (at 0 -1.43 90) (layer B.Fab)
+    (fp_text value 100nF (at 0 -1.43 90) (layer B.Fab)
       (effects (font (size 1 1) (thickness 0.15)) (justify mirror))
     )
@@
       (effects (font (size 0.5 0.5) (thickness 0.1)) (justify mirror))
     )
-    (fp_text value "10uF 25V " (at 0 -1.43 90) (layer B.Fab)
+    (fp_text value 10uF (at 0 -1.43 90) (layer B.Fab)
       (effects (font (size 1 1) (thickness 0.15)) (justify mirror))
     )
@@
       (effects (font (size 0.5 0.5) (thickness 0.1)) (justify mirror))
     )
-    (fp_text value "10uF 25V " (at 0 -1.43 90) (layer B.Fab)
+    (fp_text value 10uF (at 0 -1.43 90) (layer B.Fab)
       (effects (font (size 1 1) (thickness 0.15)) (justify mirror))
     )
@@
       (effects (font (size 0.5 0.5) (thickness 0.1)) (justify mirror))
     )
-    (fp_text value "10uF 50V " (at 0 -1.43) (layer B.Fab)
+    (fp_text value 10uF (at 0 -1.43) (layer B.Fab)
       (effects (font (size 1 1) (thickness 0.15)) (justify mirror))
     )
@@
       (effects (font (size 0.5 0.5) (thickness 0.1)) (justify mirror))
     )
-    (fp_text value "100nF 50V" (at 0 -1.43) (layer B.Fab)
+    (fp_text value 100nF (at 0 -1.43) (layer B.Fab)
       (effects (font (size 1 1) (thickness 0.15)) (justify mirror))
     )
@@
       (effects (font (size 0.5 0.5) (thickness 0.1)) (justify mirror))
     )
-    (fp_text value "100nF 50V" (at 0 -1.43 180) (layer B.Fab)
+    (fp_text value 100nF (at 0 -1.43 180) (layer B.Fab)
       (effects (font (size 1 1) (thickness 0.15)) (justify mirror))
     )
@@
       (effects (font (size 0.5 0.5) (thickness 0.1)) (justify mirror))
     )
-    (fp_text value "100nF 50V" (at 0 -1.43 180) (layer B.Fab)
+    (fp_text value 100nF (at 0 -1.43 180) (layer B.Fab)
       (effects (font (size 1 1) (thickness 0.15)) (justify mirror))
     )
@@
       (effects (font (size 0.5 0.5) (thickness 0.1)) (justify mirror))
     )
-    (fp_text value "100nF 50V" (at 0 -1.43) (layer B.Fab)
+    (fp_text value 100nF (at 0 -1.43) (layer B.Fab)
       (effects (font (size 1 1) (thickness 0.15)) (justify mirror))
     )
@@
       (net 1 GND))
     (pad 2 smd rect (at -1.33 0.65 90) (size 0.45 1.5) (layers F.Cu F.Paste F.Mask)
-      (net 16 /CAN_H))
-    (pad 1 smd rect (at -1.33 -0.65 90) (size 0.45 1.5) (layers F.Cu F.Paste F.Mask)
       (net 17 /CAN_L))
+    (pad 1 smd rect (at -1.33 -0.65 90) (size 0.45 1.5) (layers F.Cu F.Paste F.Mask)
+      (net 16 /CAN_H))
     (model ${KISYS3DMOD}/Package_TO_SOT_SMD.3dshapes/SOT-323_SC-70.wrl
       (at (xyz 0 0 0))

Commit message: manual sync with 960
Parts:
- added HS1: Heatsink, Heatsink:HEATSINK, F.Cu at (128.8, 6.66)
- added HS2: Heatsink, Heatsink:HEATSINK, F.Cu at (132.8, 6.66)
Routing:
- net /CAN_H: track 58.3 -> 57.2 mm

Commit message: V 0.2
Parts:
- removed HS1, HS2: Heatsink, Heatsink:HEATSINK
- C12, C15: value 1nF -> DNP
- J1: value Conn_01x01 -> DNP CORNER HOLE
- R12, R13, R15, R16, R17, R18, R19, R9: value 0 -> DNP
- moved R34 2.37 mm to (105.6, 31.3), turned to 0 degrees
- turned D11 to 270 degrees
- turned D17 to 180 degrees
- turned D2 to 0 degrees
- turned D5 to 270 degrees
- turned D8 to 270 degrees
- turned R14 to 90 degrees
- turned R25 to 90 degrees
- turned R28 to 90 degrees
Connections:
- D11 pad 1: /IGN_IN_1 -> Net-(D11-Pad1)
- D11 pad 2: Net-(D11-Pad2) -> /IGN_IN_1
- D17 pad 1: /CRNK_MCU -> Net-(D17-Pad1)
- D17 pad 2: Net-(D17-Pad2) -> /CRNK_MCU
- D5 pad 1: /IGN_OUT_1 -> Net-(D5-Pad1)
- D5 pad 2: Net-(D5-Pad2) -> /IGN_OUT_1
- D8 pad 1: /INJ_IN_1 -> Net-(D8-Pad1)
- D8 pad 2: Net-(D8-Pad2) -> /INJ_IN_1
- R14 pad 1: Net-(D5-Pad2) -> GND
- R14 pad 2: /V5V -> Net-(D5-Pad1)
- R25 pad 1: Net-(D8-Pad2) -> GND
- R25 pad 2: /V5V -> Net-(D8-Pad1)
- R28 pad 1: Net-(D11-Pad2) -> GND
- R28 pad 2: /V5V -> Net-(D11-Pad1)
- R34 pad 1: Net-(D17-Pad2) -> GND
- R34 pad 2: /V5V -> Net-(D17-Pad1)
Routing:
- net /V5V: track 62.8 -> 44.5 mm
- net GND: track 32.7 -> 38.5 mm, vias 247 -> 250
- net Net-(D17-Pad2): track 4.20 -> 0.00 mm
- net /CAN_H: track 57.2 -> 60.9 mm
- net /CAN_L: track 53.2 -> 56.0 mm
- net Net-(D17-Pad1): track 0.00 -> 1.72 mm
- net Net-(D8-Pad2): vias 1 -> 0
- net Net-(D8-Pad1): vias 0 -> 1
- net Net-(D5-Pad2): vias 1 -> 0
- net Net-(D5-Pad1): vias 0 -> 1
- net Net-(D11-Pad2): vias 1 -> 0
- net Net-(D11-Pad1): vias 0 -> 1
Other:
- board text added: "rusefi v0.2"
- board text removed: "rusefi v0.1"
