File: Analog_Input_Module/Analog_Input_Module.sch (KiCad schematic (older format))
At the start: 63 parts, among them J1 Conn_02x20_Odd_Even, U1 10K, U10 1.5K, U11 MCP6004, U12 10K, U13 10K, U14 10nF, U15 10nF, U16 MCP6004, U17 1K, U18 1K, U19 1.5K, U2 10K, U20 1.5K, U3 10nF, U4 10nF, U5 MCP6004, U6 MCP6004, U7 1K, U8 1K, U9 1.5K

Commit message: updated bom
Parts:
- C1, C2, C3, C4: MFG,MFG# AVX,08055C104KAT2A -> (none); VEND1,VEND1# DIGI,478-1395-1-ND -> (none)
- D1, D10, D11, D12, D13, D14, D15, D16, D2, D3, D4, D5, D6, D7, D8, D9: VEND# (none) -> 511-BAS70-04FILM
- R1, R11, R12, R15, R17, R19, R2, R20, R5, R7, R9: VEND2,VEND2# , -> (none)
- R10, R13, R14, R16, R18, R21, R22, R3, R4, R6, R8: MFG,MFG# ECG,ERA6AEB4993V -> (none); VEND1,VEND1# DIGI,P499KDACT-ND -> (none); VEND2,VEND2# , -> (none)
- U1, U12, U13, U2: VEND# (none) -> 603-YC324-JK-0710KL
- U10, U19, U20, U9: VEND# (none) -> 667-EXB-V8V152JV
- U11, U16, U5, U6: MFG,MFG# ADA4096-4ARUZ-R7 -> (none); Part # ADA4096-4ARUZ-R7 -> (none); VEND# 584-ADA4096-4ARUZ-R7 -> 579-MCP6004T-I/ST; VEND1,VEND1# DIGI,MCP6004-E/SL-ND -> (none); VEND2,VEND2# , -> (none)
- U11, U16, U5, U6: MFG,MFG# ADA4096-4ARUZ-R7 -> (none); Part # ADA4096-4ARUZ-R7 -> (none); VEND# 584-ADA4096-4ARUZ-R7 -> 579-MCP6004T-I/ST
- U14, U15, U3, U4: VEND# (none) -> 80-CA064X103K2RAUTO
- U17, U18, U7, U8: VEND# (none) -> 667-EXB-V8V102JV
