File: TLE7209_or_MC33186_H-Bridge_Breakout/TLE7209_Module.kicad_pcb (KiCad board)
At the start: 4 copper layers, 42.5 x 22 mm, 10 parts, among them J1 Conn_02x06_Odd_Even, J3 Conn_01x01, U1 TLE7209-2R

Commit message: progress
Other:
- board text added: "12V"
- board text added: "5V"
- board text added: "DIS"
- board text added: "EN"
- board text added: "GND"
- board text added: "IN1"
- board text added: "IN2"
- board text added: "OUT1"
- board text added: "OUT2"
- board text added: "SF"
- board text added: "rusefi v0.1"
Changed lines of the file:
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@@
   (general
     (thickness 1.6)
-    (drawings 4)
+    (drawings 21)
     (tracks 120)
     (zones 0)
@@
   (layers
     (0 F.Cu signal)
-    (1 PWR power hide)
+    (1 PWR power)
     (2 GND power)
     (31 B.Cu signal)
@@
     (44 Edge.Cuts user)
     (45 Margin user hide)
-    (46 B.CrtYd user)
-    (47 F.CrtYd user)
+    (46 B.CrtYd user hide)
+    (47 F.CrtYd user hide)
     (48 B.Fab user hide)
     (49 F.Fab user hide)
   )
   (setup
-    (last_trace_width 0.3048)
+    (last_trace_width 0.1524)
     (user_trace_width 0.1524)
     (user_trace_width 0.2159)
@@
     (descr "Through hole straight pin header, 2x08, 2.54mm pitch, double rows")
     (tags "Through hole pin header THT 2x08 2.54mm double row")
-    (fp_text reference J1 (at 1.27 -2.33 270) (layer F.SilkS)
+    (fp_text reference J1 (at 1.27 -2.33 270) (layer F.SilkS) hide
       (effects (font (size 1 1) (thickness 0.15)))
     )
@@
     (tags "resistor handsolder")
     (attr smd)
-    (fp_text reference R3 (at 0 -1.65 180) (layer F.SilkS)
+    (fp_text reference R3 (at 2.921 0 180) (layer F.SilkS)
       (effects (font (size 1 1) (thickness 0.15)))
     )
@@
     (tags "resistor handsolder")
     (attr smd)
-    (fp_text reference R1 (at 0 1.65 270) (layer B.SilkS)
+    (fp_text reference R1 (at -3.048 -0.127 270) (layer B.SilkS)
       (effects (font (size 1 1) (thickness 0.15)) (justify mirror))
     )
@@
     (tags "Diode SMA (DO-214AC)")
     (attr smd)
-    (fp_text reference D1 (at 0 -2.5 180) (layer F.SilkS)
+    (fp_text reference D1 (at 4.445 1.016 180) (layer F.SilkS)
       (effects (font (size 1 1) (thickness 0.15)))
     )
@@
     (tags "capacitor handsolder")
     (attr smd)
-    (fp_text reference C3 (at -3.06 -0.05 180) (layer F.SilkS)
+    (fp_text reference C3 (at 2.921 0 180) (layer F.SilkS)
       (effects (font (size 1 1) (thickness 0.15)))
     )
@@
     )
   )
+  (gr_text IN1 (at 34.29 36.322) (layer B.SilkS)
+    (effects (font (size 0.6 0.6) (thickness 0.15)) (justify mirror))
+  )
+  (gr_text 5V (at 24.13 36.322) (layer B.SilkS)
+    (effects (font (size 0.6 0.6) (thickness 0.15)) (justify mirror))
+  )
+  (gr_text GND (at 21.59 36.322) (layer B.SilkS)
+    (effects (font (size 0.6 0.6) (thickness 0.15)) (justify mirror))
+  )
+  (gr_text GND (at 21.59 35.306) (layer B.SilkS)
+    (effects (font (size 0.6 0.6) (thickness 0.15)) (justify mirror))
+  )
+  (gr_text 5V (at 24.13 35.306) (layer B.SilkS)
+    (effects (font (size 0.6 0.6) (thickness 0.15)) (justify mirror))
+  )
+  (gr_text 12V (at 26.67 36.322) (layer B.SilkS)
+    (effects (font (size 0.6 0.6) (thickness 0.15)) (justify mirror))
+  )
+  (gr_text 12V (at 26.67 35.306) (layer B.SilkS)
+    (effects (font (size 0.6 0.6) (thickness 0.15)) (justify mirror))
+  )
+  (gr_text IN2 (at 29.464 36.322) (layer B.SilkS)
+    (effects (font (size 0.6 0.6) (thickness 0.15)) (justify mirror))
+  )
+  (gr_text EN (at 29.464 35.306) (layer B.SilkS)
+    (effects (font (size 0.6 0.6) (thickness 0.15)) (justify mirror))
+  )
+  (gr_text DIS (at 32.004 35.306) (layer B.SilkS)
+    (effects (font (size 0.6 0.6) (thickness 0.15)) (justify mirror))
+  )
+  (gr_text SF (at 34.29 35.306) (layer B.SilkS)
+    (effects (font (size 0.6 0.6) (thickness 0.15)) (justify mirror))
+  )
+  (gr_text OUT2 (at 37.084 36.322) (layer B.SilkS)
+    (effects (font (size 0.6 0.6) (thickness 0.15)) (justify mirror))
+  )
+  (gr_text OUT2 (at 37.084 35.306) (layer B.SilkS)
+    (effects (font (size 0.6 0.6) (thickness 0.15)) (justify mirror))
+  )
+  (gr_text "OUT1\n" (at 39.878 35.306) (layer B.SilkS)
+    (effects (font (size 0.6 0.6) (thickness 0.15)) (justify mirror))
+  )
+  (gr_text "OUT1\n" (at 39.878 36.322) (layer B.SilkS)
+    (effects (font (size 0.6 0.6) (thickness 0.15)) (justify mirror))
+  )
+  (gr_circle (center 46.228 37.846) (end 46.736 38.354) (layer F.SilkS) (width 0.25))
+  (gr_text "rusefi v0.1" (at 30.226 22.606) (layer F.SilkS)
+    (effects (font (size 1 1) (thickness 0.15)))
+  )
   (gr_line (start 62.484 20) (end 20 20) (layer Edge.Cuts) (width 0.15))

Commit message: progress
Parts:
- added R4: 10K, Resistor_SMD:R_0805_2012Metric_Pad1.15x1.40mm_HandSolder, B.Cu at (33.3, 28.2)
- added R5: 10K, Resistor_SMD:R_0805_2012Metric_Pad1.15x1.40mm_HandSolder, B.Cu at (41.4, 27.4)
- moved R2 0.21 mm to (52.6, 40.1)
- moved C1 0.13 mm to (28.2, 30.2)
Routing:
- net /EN: track 38.2 -> 40.4 mm
- net /DIS: track 28.2 -> 29.3 mm
- net /5V: track 34.6 -> 35.6 mm, vias 1 -> 2
Other:
- board size 42.5 x 22 mm -> 43 x 22 mm

Commit message: sync
Parts:
- R5: moved to F.Cu
- moved R5 7.60 mm to (34.1, 25.3)
- moved R4 6.04 mm to (27.4, 26.9)
- moved R1 1.75 mm to (42.4, 36.1)
- moved C3 0.76 mm to (38.2, 31.8)
- moved R3 0.45 mm to (38.2, 33.7)
Connections:
- J1 pad 10: /IN2 -> Net-(J1-Pad10)
- J1 pad 7: /DIS -> /IN2
- J1 pad 8: Net-(J1-Pad8) -> /DIS
Routing:
- net Net-(C1-Pad1): track 9.91 -> 51.0 mm
- net /DIS: track 29.3 -> 40.2 mm, vias 1 -> 2
- net /EN: track 40.4 -> 45.4 mm
- net /IN2: track 30.8 -> 34.1 mm
- net /OUT1: track 31.5 -> 34.2 mm
- net /SF: track 19.7 -> 22.3 mm
- net /5V: track 35.6 -> 36.5 mm
- net GND: vias 4 -> 118
- removed copper zone on GND, net GND
- removed copper zone on PWR, net Net-(C1-Pad1)
Other:
- copper layers 4 -> 2
- board text added: "TLE7209"

Commit message: sync
Connections:
- J1 pad 10: Net-(J1-Pad10) -> /DIS
- J1 pad 8: /DIS -> Net-(J1-Pad8)
Routing:
- net GND: track 0.00 -> 11.2 mm, vias 118 -> 391

Commit message: Pcb Update
Parts:
- added C4: CP1, Capacitor_SMD:CP_Elec_6.3x5.7, F.Cu at (31.5, 24.7)
- C2, R1, R2, R4: moved to F.Cu
- moved R4 6.83 mm to (32.7, 31.1), turned to 270 degrees
- moved R5 5.86 mm to (34.7, 31.2)
- moved D1 4.49 mm to (24.1, 32.4)
- moved C2 3.56 mm to (54.6, 40.8)
- moved R2 3.08 mm to (49.6, 40.8), turned to 0 degrees
- moved C1 2.59 mm to (28.7, 32.8), turned to 270 degrees
- moved U1 0.96 mm to (53.9, 29.9)
- moved R1 0.33 mm to (42.7, 36.0)
Connections:
- C1 pad 1: Net-(C1-Pad1) -> /12V
- C1 pad 2: /12V -> GND
- C2 pad 1: Net-(C1-Pad1) -> /12V
- D1 pad 1: Net-(C1-Pad1) -> /12V
- D1 pad 2: /12V -> GND
- R2 pad 1: Net-(C1-Pad1) -> /12V
- U1 pad 16: Net-(C1-Pad1) -> /12V
- U1 pad 5: Net-(C1-Pad1) -> /12V
Routing:
- net /12V: track 10.8 -> 85.7 mm, vias 1 -> 6
- net Net-(C1-Pad1): track 51.0 -> 0.00 mm, vias 3 -> 0
- net Net-(C2-Pad2): track 4.69 -> 9.51 mm, vias 1 -> 2
- net /5V: track 36.5 -> 34.3 mm, vias 2 -> 3
- net /EN: track 45.4 -> 47.4 mm, vias 1 -> 2
- net /DIS: track 40.1 -> 41.3 mm
- net /IN2: track 34.1 -> 33.2 mm
- net /IN1: track 19.5 -> 20.0 mm
- net /OUT2: track 39.6 -> 40.2 mm
- net /SF: vias 1 -> 2
- net GND: vias 391 -> 272
Other:
- board text added: "rusefi v0.2"
- board text removed: "TLE7209"
- board text removed: "rusefi v0.1"

Commit message: Gerbers
Routing:
- net GND: vias 272 -> 271
Changed lines of the file:
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@@
     (thickness 1.6)
     (drawings 36)
-    (tracks 477)
+    (tracks 476)
     (zones 0)
     (modules 13)
@@
   (via (at 46.0502 40.5892) (size 0.6) (drill 0.3) (layers F.Cu B.Cu) (net 1))
   (via (at 44.7802 40.5892) (size 0.6) (drill 0.3) (layers F.Cu B.Cu) (net 1))
-  (via (at 43.5102 40.5892) (size 0.6) (drill 0.3) (layers F.Cu B.Cu) (net 1))
   (via (at 42.2402 40.5892) (size 0.6) (drill 0.3) (layers F.Cu B.Cu) (net 1))
   (via (at 41.6052 40.5892) (size 0.6) (drill 0.3) (layers F.Cu B.Cu) (net 1))

Commit message: version (#27)
Parts:
- C4: footprint Capacitor_SMD:CP_Elec_6.3x5.7 -> Capacitor_SMD:CP_Elec_8x10
Routing:
- net GND: vias 271 -> 266
Changed lines of the file:
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@@
     (thickness 1.6)
     (drawings 36)
-    (tracks 476)
+    (tracks 471)
     (zones 0)
     (modules 13)
@@
     (title "TLE7209-2R Module")
     (date 2019-01-31)
-    (rev R0.1)
+    (rev R0.2)
   )
   (layers
@@
     (uvia_drill 0.127)
   )
+  (module Capacitor_SMD:CP_Elec_8x10 (layer F.Cu)
+    (at 31.5468 24.7142)
+    (descr "SMD capacitor, aluminum electrolytic, Nichicon, 8.0x10mm")
+    (tags "capacitor electrolytic")
+    (attr smd)
+    (fp_text reference C4 (at -5.588 3.1242) (layer F.SilkS)
+      (effects (font (size 1 1) (thickness 0.15)))
+    )
+    (fp_text value CP1 (at 0 5.2) (layer F.Fab)
+      (effects (font (size 1 1) (thickness 0.15)))
+    )
+    (fp_text user %R (at 0 0) (layer F.Fab)
+      (effects (font (size 1 1) (thickness 0.15)))
+    )
+    (fp_line (start -5.25 1.5) (end -4.4 1.5) (layer F.CrtYd) (width 0.05))
+    (fp_line (start -5.25 -1.5) (end -5.25 1.5) (layer F.CrtYd) (width 0.05))
+    (fp_line (start -4.4 -1.5) (end -5.25 -1.5) (layer F.CrtYd) (width 0.05))
+    (fp_line (start -4.4 1.5) (end -4.4 3.25) (layer F.CrtYd) (width 0.05))
+    (fp_line (start -4.4 -3.25) (end -4.4 -1.5) (layer F.CrtYd) (width 0.05))
+    (fp_line (start -4.4 -3.25) (end -3.25 -4.4) (layer F.CrtYd) (width 0.05))
+    (fp_line (start -4.4 3.25) (end -3.25 4.4) (layer F.CrtYd) (width 0.05))
+    (fp_line (start -3.25 -4.4) (end 4.4 -4.4) (layer F.CrtYd) (width 0.05))
+    (fp_line (start -3.25 4.4) (end 4.4 4.4) (layer F.CrtYd) (width 0.05))
+    (fp_line (start 4.4 1.5) (end 4.4 4.4) (layer F.CrtYd) (width 0.05))
+    (fp_line (start 5.25 1.5) (end 4.4 1.5) (layer F.CrtYd) (width 0.05))
+    (fp_line (start 5.25 -1.5) (end 5.25 1.5) (layer F.CrtYd) (width 0.05))
+    (fp_line (start 4.4 -1.5) (end 5.25 -1.5) (layer F.CrtYd) (width 0.05))
+    (fp_line (start 4.4 -4.4) (end 4.4 -1.5) (layer F.CrtYd) (width 0.05))
+    (fp_line (start -5 -3.01) (end -5 -2.01) (layer F.SilkS) (width 0.12))
+    (fp_line (start -5.5 -2.51) (end -4.5 -2.51) (layer F.SilkS) (width 0.12))
+    (fp_line (start -4.26 3.195563) (end -3.195563 4.26) (layer F.SilkS) (width 0.12))
+    (fp_line (start -4.26 -3.195563) (end -3.195563 -4.26) (layer F.SilkS) (width 0.12))
+    (fp_line (start -4.26 -3.195563) (end -4.26 -1.51) (layer F.SilkS) (width 0.12))
+    (fp_line (start -4.26 3.195563) (end -4.26 1.51) (layer F.SilkS) (width 0.12))
+    (fp_line (start -3.195563 4.26) (end 4.26 4.26) (layer F.SilkS) (width 0.12))
+    (fp_line (start -3.195563 -4.26) (end 4.26 -4.26) (layer F.SilkS) (width 0.12))
+    (fp_line (start 4.26 -4.26) (end 4.26 -1.51) (layer F.SilkS) (width 0.12))
+    (fp_line (start 4.26 4.26) (end 4.26 1.51) (layer F.SilkS) (width 0.12))
+    (fp_line (start -3.162278 -1.9) (end -3.162278 -1.1) (layer F.Fab) (width 0.1))
+    (fp_line (start -3.562278 -1.5) (end -2.762278 -1.5) (layer F.Fab) (width 0.1))
+    (fp_line (start -4.15 3.15) (end -3.15 4.15) (layer F.Fab) (width 0.1))
+    (fp_line (start -4.15 -3.15) (end -3.15 -4.15) (layer F.Fab) (width 0.1))
+    (fp_line (start -4.15 -3.15) (end -4.15 3.15) (layer F.Fab) (width 0.1))
+    (fp_line (start -3.15 4.15) (end 4.15 4.15) (layer F.Fab) (width 0.1))
+    (fp_line (start -3.15 -4.15) (end 4.15 -4.15) (layer F.Fab) (width 0.1))
+    (fp_line (start 4.15 -4.15) (end 4.15 4.15) (layer F.Fab) (width 0.1))
+    (fp_circle (center 0 0) (end 4 0) (layer F.Fab) (width 0.1))
+    (pad 2 smd roundrect (at 3.25 0) (size 3.5 2.5) (layers F.Cu F.Paste F.Mask) (roundrect_rratio 0.1)
+      (net 1 GND))
+    (pad 1 smd roundrect (at -3.25 0) (size 3.5 2.5) (layers F.Cu F.Paste F.Mask) (roundrect_rratio 0.1)
+      (net 5 /12V))
+    (model ${KISYS3DMOD}/Capacitor_SMD.3dshapes/CP_Elec_8x10.wrl
+      (at (xyz 0 0 0))
+      (scale (xyz 1 1 1))
+      (rotate (xyz 0 0 0))
+    )
+  )
   (module Package_SO:HSOP-20-1EP_11.0x15.9mm_P1.27mm_SlugDown_ThermalVias (layer F.Cu)
     (at 53.9242 29.9212 90)
@@
       (at (xyz 0 0 0))
       (scale (xyz 2.2 1.95 2))
-      (rotate (xyz 0 0 0))
-    )
-  )
-  (module Capacitor_SMD:CP_Elec_6.3x5.7 (layer F.Cu)
-    (at 31.5468 24.7142)
-    (descr "SMD capacitor, aluminum electrolytic, United Chemi-Con, 6.3x5.7mm")
-    (tags "capacitor electrolytic")
-    (attr smd)
-    (fp_text reference C4 (at 4.8768 2.3368) (layer F.SilkS)
-      (effects (font (size 1 1) (thickness 0.15)))
-    )
-    (fp_text value CP1 (at 0 4.35) (layer F.Fab)
-      (effects (font (size 1 1) (thickness 0.15)))
-    )
-    (fp_text user %R (at 0 0) (layer F.Fab)
-      (effects (font (size 1 1) (thickness 0.15)))
-    )
-    (fp_line (start -4.7 1.05) (end -3.55 1.05) (layer F.CrtYd) (width 0.05))
-    (fp_line (start -4.7 -1.05) (end -4.7 1.05) (layer F.CrtYd) (width 0.05))
-    (fp_line (start -3.55 -1.05) (end -4.7 -1.05) (layer F.CrtYd) (width 0.05))
-    (fp_line (start -3.55 1.05) (end -3.55 2.4) (layer F.CrtYd) (width 0.05))
-    (fp_line (start -3.55 -2.4) (end -3.55 -1.05) (layer F.CrtYd) (width 0.05))
-    (fp_line (start -3.55 -2.4) (end -2.4 -3.55) (layer F.CrtYd) (width 0.05))
-    (fp_line (start -3.55 2.4) (end -2.4 3.55) (layer F.CrtYd) (width 0.05))
-    (fp_line (start -2.4 -3.55) (end 3.55 -3.55) (layer F.CrtYd) (width 0.05))
-    (fp_line (start -2.4 3.55) (end 3.55 3.55) (layer F.CrtYd) (width 0.05))
-    (fp_line (start 3.55 1.05) (end 3.55 3.55) (layer F.CrtYd) (width 0.05))
-    (fp_line (start 4.7 1.05) (end 3.55 1.05) (layer F.CrtYd) (width 0.05))
-    (fp_line (start 4.7 -1.05) (end 4.7 1.05) (layer F.CrtYd) (width 0.05))
-    (fp_line (start 3.55 -1.05) (end 4.7 -1.05) (layer F.CrtYd) (width 0.05))
-    (fp_line (start 3.55 -3.55) (end 3.55 -1.05) (layer F.CrtYd) (width 0.05))
-    (fp_line (start -4.04375 -2.24125) (end -4.04375 -1.45375) (layer F.SilkS) (width 0.12))
-    (fp_line (start -4.4375 -1.8475) (end -3.65 -1.8475) (layer F.SilkS) (width 0.12))
-    (fp_line (start -3.41 2.345563) (end -2.345563 3.41) (layer F.SilkS) (width 0.12))
-    (fp_line (start -3.41 -2.345563) (end -2.345563 -3.41) (layer F.SilkS) (width 0.12))
-    (fp_line (start -3.41 -2.345563) (end -3.41 -1.06) (layer F.SilkS) (width 0.12))
-    (fp_line (start -3.41 2.345563) (end -3.41 1.06) (layer F.SilkS) (width 0.12))
-    (fp_line (start -2.345563 3.41) (end 3.41 3.41) (layer F.SilkS) (width 0.12))
-    (fp_line (start -2.345563 -3.41) (end 3.41 -3.41) (layer F.SilkS) (width 0.12))
-    (fp_line (start 3.41 -3.41) (end 3.41 -1.06) (layer F.SilkS) (width 0.12))
-    (fp_line (start 3.41 3.41) (end 3.41 1.06) (layer F.SilkS) (width 0.12))
-    (fp_line (start -2.389838 -1.645) (end -2.389838 -1.015) (layer F.Fab) (width 0.1))
-    (fp_line (start -2.704838 -1.33) (end -2.074838 -1.33) (layer F.Fab) (width 0.1))
-    (fp_line (start -3.3 2.3) (end -2.3 3.3) (layer F.Fab) (width 0.1))
-    (fp_line (start -3.3 -2.3) (end -2.3 -3.3) (layer F.Fab) (width 0.1))
-    (fp_line (start -3.3 -2.3) (end -3.3 2.3) (layer F.Fab) (width 0.1))
-    (fp_line (start -2.3 3.3) (end 3.3 3.3) (layer F.Fab) (width 0.1))
-    (fp_line (start -2.3 -3.3) (end 3.3 -3.3) (layer F.Fab) (width 0.1))
-    (fp_line (start 3.3 -3.3) (end 3.3 3.3) (layer F.Fab) (width 0.1))
-    (fp_circle (center 0 0) (end 3.15 0) (layer F.Fab) (width 0.1))
-    (pad 2 smd roundrect (at 2.7 0) (size 3.5 1.6) (layers F.Cu F.Paste F.Mask) (roundrect_rratio 0.15625)
-      (net 1 GND))
-    (pad 1 smd roundrect (at -2.7 0) (size 3.5 1.6) (layers F.Cu F.Paste F.Mask) (roundrect_rratio 0.15625)
-      (net 5 /12V))
-    (model ${KISYS3DMOD}/Capacitor_SMD.3dshapes/CP_Elec_6.3x5.7.wrl
-      (at (xyz 0 0 0))
-      (scale (xyz 1 1 1))
       (rotate (xyz 0 0 0))
     )
@@
   (via (at 37.4904 24.4602) (size 0.6) (drill 0.3) (layers F.Cu B.Cu) (net 1))
   (via (at 37.0332 25.0952) (size 0.6) (drill 0.3) (layers F.Cu B.Cu) (net 1))
-  (via (at 35.9664 26.2636) (size 0.6) (drill 0.3) (layers F.Cu B.Cu) (net 1))
   (via (at 35.2044 27.0256) (size 0.6) (drill 0.3) (layers F.Cu B.Cu) (net 1))
   (via (at 34.4678 27.8638) (size 0.6) (drill 0.3) (layers F.Cu B.Cu) (net 1))
@@
   (via (at 32.004 21.844) (size 0.78994) (drill 0.43434) (layers F.Cu B.Cu) (net 1))
   (via (at 33.02 21.844) (size 0.78994) (drill 0.43434) (layers F.Cu B.Cu) (net 1))
-  (via (at 26.924 22.86) (size 0.78994) (drill 0.43434) (layers F.Cu B.Cu) (net 1))
-  (via (at 27.94 22.86) (size 0.78994) (drill 0.43434) (layers F.Cu B.Cu) (net 1))
-  (via (at 28.956 22.86) (size 0.78994) (drill 0.43434) (layers F.Cu B.Cu) (net 1))
-  (via (at 29.972 22.86) (size 0.78994) (drill 0.43434) (layers F.Cu B.Cu) (net 1))
   (via (at 30.988 22.86) (size 0.78994) (drill 0.43434) (layers F.Cu B.Cu) (net 1))
   (via (at 32.004 22.86) (size 0.78994) (drill 0.43434) (layers F.Cu B.Cu) (net 1))
