File: lowside/lowside.kicad_pcb (KiCad board)
At the start: 4 copper layers, 101 x 22 mm, 348 parts, among them J1 Conn_02x39_Odd_Even, U1 VNLD5090, U2 VNLD5090, U3 VNLD5090, U4 VNLD5090, U5 VNLD5090, U6 VNLD5090, U7 VNLD5090

Commit message: Generated gerbers and BOM for MFG.
Other:
- rule pad_to_mask_clearance: 0.051 -> 0.0762
Changed lines of the file:
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@@
     (pad_size 0.6 0.6)
     (pad_drill 0.3)
-    (pad_to_mask_clearance 0.051)
-    (solder_mask_min_width 0.25)
+    (pad_to_mask_clearance 0.0762)
     (aux_axis_origin 0 0)
     (visible_elements 7FFFFFFF)
@@
       (outputformat 1)
       (mirror false)
-      (drillshape 1)
+      (drillshape 0)
       (scaleselection 1)
-      (outputdirectory ""))
+      (outputdirectory "gerbers/"))
   )
   (net 0 "")
