File: lowside/pair.sch (KiCad schematic (older format))
At the start: 13 parts, among them U1 VNLD5090

Commit message: Generated gerbers and BOM for MFG.
Parts:
- D1, D2: MFG,MFG# LITTELFUSE,TPSMF4L36A -> DIODES_INC,SBR2U60S1F; Vend1,Vend1# DIGI,F7526CT-ND -> DIGI,SBR2U60S1F-7DICT-ND
Changed lines of the file:
@@
 Sheet 2 8
 Title ""
-Date ""
-Rev ""
-Comp ""
+Date "2020-02-15"
+Rev "R0.1"
+Comp "rusEFI"
 Comment1 ""
 Comment2 ""
@@
 F 2 "Diode_SMD:D_SMF" H 4250 1250 50  0001 C CNN
 F 3 "~" H 4250 1250 50  0001 C CNN
-F 4 "LITTELFUSE,TPSMF4L36A" H 4250 1250 50  0001 C CNN "MFG,MFG#"
-F 5 "DIGI,F7526CT-ND" H 4250 1250 50  0001 C CNN "Vend1,Vend1#"
+F 4 "DIODES_INC,SBR2U60S1F" H 4250 1250 50  0001 C CNN "MFG,MFG#"
+F 5 "DIGI,SBR2U60S1F-7DICT-ND" H 4250 1250 50  0001 C CNN "Vend1,Vend1#"
 	1    4250 1250
 	0    1    1    0
@@
 F 2 "Diode_SMD:D_SMF" H 4250 2300 50  0001 C CNN
 F 3 "~" H 4250 2300 50  0001 C CNN
-F 4 "LITTELFUSE,TPSMF4L36A" H 4250 2300 50  0001 C CNN "MFG,MFG#"
-F 5 "DIGI,F7526CT-ND" H 4250 2300 50  0001 C CNN "Vend1,Vend1#"
+F 4 "DIODES_INC,SBR2U60S1F" H 4250 2300 50  0001 C CNN "MFG,MFG#"
+F 5 "DIGI,SBR2U60S1F-7DICT-ND" H 4250 2300 50  0001 C CNN "Vend1,Vend1#"
 	1    4250 2300
 	0    -1   -1   0

Commit message: getting ready for assembly
Parts:
- C1, C2: LCSC (none) -> C81355
- D1, D2: LCSC (none) -> C156309
- D15, D16: LCSC (none) -> C2286
- R1, R2, R23, R24: LCSC (none) -> C21190
- R3, R4: LCSC (none) -> C25804
- U1: LCSC (none) -> C222209
Connections:
- net +12V: now also R24.1; no longer R24.2
- net at D16.2 (A): now also R24.2; no longer R24.1
Changed lines of the file:
@@
 EESchema Schematic File Version 4
-EELAYER 30 0
+LIBS:lowside-cache
+EELAYER 29 0
 EELAYER END
 $Descr A4 11693 8268
 encoding utf-8
-Sheet 2 8
+Sheet 3 8
 Title ""
 Date "2020-02-15"
@@
 AR Path="/5E2D1A0F/5E28FEFB" Ref="U6"  Part="1"
 AR Path="/5E2B6330/5E28FEFB" Ref="U7"  Part="1"
-F 0 "U1" H 3100 2547 60  0000 C CNN
+F 0 "U2" H 3100 2547 60  0000 C CNN
 F 1 "VNLD5090" H 3100 2441 60  0000 C CNN
 F 2 "Package_SO:SO-8_3.9x4.9mm_P1.27mm" H 3200 1650 60  0001 C CNN
@@
 F 4 "ST,VNLD5090TR-E" H 3100 1900 50  0001 C CNN "MFG,MFG#"
 F 5 "DIGI,497-14323-1-ND" H 3100 1900 50  0001 C CNN "Vend1,Vend1#"
+F 6 "C222209" H 3100 1900 50  0001 C CNN "LCSC"
 	1    3100 1900
 	1    0    0    -1
@@
 AR Path="/5E2D1A0F/5E290D55" Ref="#PWR0163"  Part="1"
 AR Path="/5E2B6330/5E290D55" Ref="#PWR0177"  Part="1"
-F 0 "#PWR0113" H 3300 2250 50  0001 C CNN
+F 0 "#PWR0119" H 3300 2250 50  0001 C CNN
 F 1 "GND" H 3305 2327 50  0000 C CNN
 F 2 "" H 3300 2500 50  0001 C CNN
@@
 AR Path="/5E2D1A0F/5E291066" Ref="#PWR0164"  Part="1"
 AR Path="/5E2B6330/5E291066" Ref="#PWR0178"  Part="1"
-F 0 "#PWR0114" H 3400 2250 50  0001 C CNN
+F 0 "#PWR0120" H 3400 2250 50  0001 C CNN
 F 1 "GND" H 3405 2327 50  0000 C CNN
 F 2 "" H 3400 2500 50  0001 C CNN
@@
 AR Path="/5E2D1A0F/5E291CC1" Ref="R31"  Part="1"
 AR Path="/5E2B6330/5E291CC1" Ref="R39"  Part="1"
-F 0 "R1" V 2100 1500 50  0000 C CNN
+F 0 "R5" V 2100 1500 50  0000 C CNN
 F 1 "1k" V 2200 1500 50  0000 C CNN
 F 2 "Resistor_SMD:R_0603_1608Metric" V 2130 1500 50  0001 C CNN
@@
 F 4 "YAGEO,RC0603JR-071KL" H 2200 1500 50  0001 C CNN "MFG,MFG#"
 F 5 "DIGI,311-1.0KGRCT-ND" H 2200 1500 50  0001 C CNN "Vend1,Vend1#"
+F 6 "C21190" V 2200 1500 50  0001 C CNN "LCSC"
 	1    2200 1500
 	0    1    1    0
@@
 AR Path="/5E2D1A0F/5E292256" Ref="R32"  Part="1"
 AR Path="/5E2B6330/5E292256" Ref="R40"  Part="1"
-F 0 "R2" V 2300 2050 50  0000 C CNN
+F 0 "R6" V 2300 2050 50  0000 C CNN
 F 1 "1k" V 2200 2050 50  0000 C CNN
 F 2 "Resistor_SMD:R_0603_1608Metric" V 2130 2050 50  0001 C CNN
@@
 F 4 "YAGEO,RC0603JR-071KL" H 2200 2050 50  0001 C CNN "MFG,MFG#"
 F 5 "DIGI,311-1.0KGRCT-ND" H 2200 2050 50  0001 C CNN "Vend1,Vend1#"
+F 6 "C21190" V 2200 2050 50  0001 C CNN "LCSC"
 	1    2200 2050
 	0    1    1    0
@@
 AR Path="/5E2D1A0F/5E2928C2" Ref="C11"  Part="1"
 AR Path="/5E2B6330/5E2928C2" Ref="C13"  Part="1"
-F 0 "C1" H 3635 1204 50  0000 R CNN
+F 0 "C3" H 3635 1204 50  0000 R CNN
 F 1 "6.8n" H 3635 1295 50  0000 R CNN
 F 2 "Capacitor_SMD:C_0603_1608Metric" H 3788 1100 50  0001 C CNN
@@
 F 4 "KE MET,C0603C682K1RACTU" H 3750 1250 50  0001 C CNN "MFG,MFG#"
 F 5 "DIGI,399-3187-1-ND" H 3750 1250 50  0001 C CNN "Vend1,Vend1#"
+F 6 "C81355" H 3750 1250 50  0001 C CNN "LCSC"
 	1    3750 1250
 	-1   0    0    1
@@
 AR Path="/5E2D1A0F/5E293060" Ref="C12"  Part="1"
 AR Path="/5E2B6330/5E293060" Ref="C14"  Part="1"
-F 0 "C2" H 3865 2346 50  0000 L CNN
+F 0 "C4" H 3865 2346 50  0000 L CNN
 F 1 "6.8n" H 3865 2255 50  0000 L CNN
 F 2 "Capacitor_SMD:C_0603_1608Metric" H 3788 2150 50  0001 C CNN
@@
 F 4 "KE MET,C0603C682K1RACTU" H 3750 2300 50  0001 C CNN "MFG,MFG#"
 F 5 "DIGI,399-3187-1-ND" H 3750 2300 50  0001 C CNN "Vend1,Vend1#"
+F 6 "C81355" H 3750 2300 50  0001 C CNN "LCSC"
 	1    3750 2300
 	1    0    0    -1
@@
 AR Path="/5E2D1A0F/5E293508" Ref="#PWR0165"  Part="1"
 AR Path="/5E2B6330/5E293508" Ref="#PWR0179"  Part="1"
-F 0 "#PWR0115" H 3750 850 50  0001 C CNN
+F 0 "#PWR0121" H 3750 850 50  0001 C CNN
 F 1 "GND" H 3755 927 50  0000 C CNN
 F 2 "" H 3750 1100 50  0001 C CNN
@@
 AR Path="/5E2D1A0F/5E294C43" Ref="#PWR0166"  Part="1"
 AR Path="/5E2B6330/5E294C43" Ref="#PWR0180"  Part="1"
-F 0 "#PWR0116" H 3750 2200 50  0001 C CNN
+F 0 "#PWR0122" H 3750 2200 50  0001 C CNN
 F 1 "GND" H 3755 2277 50  0000 C CNN
 F 2 "" H 3750 2450 50  0001 C CNN
@@
 AR Path="/5E2D1A0F/5E295706" Ref="#PWR0167"  Part="1"
 AR Path="/5E2B6330/5E295706" Ref="#PWR0181"  Part="1"
-F 0 "#PWR0117" H 2450 2350 50  0001 C CNN
+F 0 "#PWR0123" H 2450 2350 50  0001 C CNN
 F 1 "GND" H 2455 2427 50  0000 C CNN
 F 2 "" H 2450 2600 50  0001 C CNN
@@
 AR Path="/5E2D1A0F/5E295C01" Ref="R34"  Part="1"
 AR Path="/5E2B6330/5E295C01" Ref="R42"  Part="1"
-F 0 "R4" V 2350 2400 50  0000 L CNN
+F 0 "R8" V 2350 2400 50  0000 L CNN
 F 1 "10k" V 2450 2350 50  0000 L CNN
 F 2 "Resistor_SMD:R_0603_1608Metric" V 2380 2450 50  0001 C CNN
@@
 F 4 "YAGEO,RC0603JR-0710KL" H 2450 2450 50  0001 C CNN "MFG,MFG#"
 F 5 "DIGI,311-10KGRCT-ND" H 2450 2450 50  0001 C CNN "Vend1,Vend1#"
+F 6 "C25804" V 2450 2450 50  0001 C CNN "LCSC"
 	1    2450 2450
 	1    0    0    -1
@@
 AR Path="/5E2D1A0F/5E295EF2" Ref="R33"  Part="1"
 AR Path="/5E2B6330/5E295EF2" Ref="R41"  Part="1"
-F 0 "R3" V 2550 1200 50  0000 L CNN
+F 0 "R7" V 2550 1200 50  0000 L CNN
 F 1 "10k" V 2450 1200 50  0000 L CNN
 F 2 "Resistor_SMD:R_0603_1608Metric" V 2380 1250 50  0001 C CNN
@@
 F 4 "YAGEO,RC0603JR-0710KL" H 2450 1250 50  0001 C CNN "MFG,MFG#"
 F 5 "DIGI,311-10KGRCT-ND" H 2450 1250 50  0001 C CNN "Vend1,Vend1#"
+F 6 "C25804" V 2450 1250 50  0001 C CNN "LCSC"
 	1    2450 1250
 	-1   0    0    1
@@
 AR Path="/5E2D1A0F/5E297A73" Ref="#PWR0168"  Part="1"
 AR Path="/5E2B6330/5E297A73" Ref="#PWR0182"  Part="1"
-F 0 "#PWR0118" H 2450 850 50  0001 C CNN
+F 0 "#PWR0124" H 2450 850 50  0001 C CNN
 F 1 "GND" H 2455 927 50  0000 C CNN
 F 2 "" H 2450 1100 50  0001 C CNN
@@
 AR Path="/5E2D1A0F/5E2A21C5" Ref="D21"  Part="1"
 AR Path="/5E2B6330/5E2A21C5" Ref="D27"  Part="1"
-F 0 "D1" V 4204 1329 50  0000 L CNN
+F 0 "D3" V 4204 1329 50  0000 L CNN
 F 1 "D_Schottky" V 4295 1329 50  0000 L CNN
 F 2 "Diode_SMD:D_SMF" H 4250 1250 50  0001 C CNN
@@
 F 4 "DIODES_INC,SBR2U60S1F" H 4250 1250 50  0001 C CNN "MFG,MFG#"
 F 5 "DIGI,SBR2U60S1F-7DICT-ND" H 4250 1250 50  0001 C CNN "Vend1,Vend1#"
+F 6 "C156309" V 4250 1250 50  0001 C CNN "LCSC"
 	1    4250 1250
 	0    1    1    0
@@
 AR Path="/5E2D1A0F/5E2A29A5" Ref="#PWR0169"  Part="1"
 AR Path="/5E2B6330/5E2A29A5" Ref="#PWR0183"  Part="1"
-F 0 "#PWR0137" H 4250 950 50  0001 C CNN
+F 0 "#PWR0139" H 4250 950 50  0001 C CNN
 F 1 "+12V" H 4265 1273 50  0000 C CNN
 F 2 "" H 4250 1100 50  0001 C CNN
@@
 AR Path="/5E2D1A0F/5E2A30AB" Ref="D22"  Part="1"
 AR Path="/5E2B6330/5E2A30AB" Ref="D28"  Part="1"
-F 0 "D2" V 4296 2221 50  0000 R CNN
+F 0 "D4" V 4296 2221 50  0000 R CNN
 F 1 "D_Schottky" V 4205 2221 50  0000 R CNN
 F 2 "Diode_SMD:D_SMF" H 4250 2300 50  0001 C CNN
@@
 F 4 "DIODES_INC,SBR2U60S1F" H 4250 2300 50  0001 C CNN "MFG,MFG#"
 F 5 "DIGI,SBR2U60S1F-7DICT-ND" H 4250 2300 50  0001 C CNN "Vend1,Vend1#"
+F 6 "C156309" V 4250 2300 50  0001 C CNN "LCSC"
 	1    4250 2300
 	0    -1   -1   0
@@
 AR Path="/5E2D1A0F/5E2A3E5A" Ref="#PWR0170"  Part="1"
 AR Path="/5E2B6330/5E2A3E5A" Ref="#PWR0184"  Part="1"
-F 0 "#PWR0138" H 4250 2300 50  0001 C CNN
+F 0 "#PWR0140" H 4250 2300 50  0001 C CNN
 F 1 "+12V" H 4265 2623 50  0000 C CNN
 F 2 "" H 4250 2450 50  0001 C CNN
@@
 AR Path="/5E2D1A0F/5E2BF0E5" Ref="D24"  Part="1"
 AR Path="/5E2B6330/5E2BF0E5" Ref="D30"  Part="1"
-F 0 "D10" V 4897 2378 50  0000 L CNN
+F 0 "D12" V 4897 2378 50  0000 L CNN
 F 1 "LED" V 4988 2378 50  0000 L CNN
 F 2 "LED_SMD:LED_0603_1608Metric" H 4950 2300 50  0001 C CNN
@@
 F 4 "DIALIGHT,598-8010-107F" H 4950 2300 50  0001 C CNN "MFG,MFG#"
 F 5 "DIGI,350-2029-1-ND" H 4950 2300 50  0001 C CNN "Vend1,Vend1#"
+F 6 "C2286" V 4950 2300 50  0001 C CNN "LCSC"
 	1    4950 2300
 	0    1    1    0
@@
 AR Path="/5E2D1A0F/5E2C027A" Ref="#PWR0171"  Part="1"
 AR Path="/5E2B6330/5E2C027A" Ref="#PWR0185"  Part="1"
-F 0 "#PWR0145" H 4950 2600 50  0001 C CNN
+F 0 "#PWR0147" H 4950 2600 50  0001 C CNN
 F 1 "+12V" H 4965 2923 50  0000 C CNN
 F 2 "" H 4950 2750 50  0001 C CNN
@@
 AR Path="/5E2D1A0F/5E2C0BF3" Ref="R36"  Part="1"
 AR Path="/5E2B6330/5E2C0BF3" Ref="R44"  Part="1"
-F 0 "R18" H 5020 2646 50  0000 L CNN
+F 0 "R20" H 5020 2646 50  0000 L CNN
 F 1 "1k" H 5020 2555 50  0000 L CNN
 F 2 "Resistor_SMD:R_0603_1608Metric" V 4880 2600 50  0001 C CNN
@@
 F 4 "YAGEO,RC0603JR-071KL" H 4950 2600 50  0001 C CNN "MFG,MFG#"
 F 5 "DIGI,311-1.0KGRCT-ND" H 4950 2600 50  0001 C CNN "Vend1,Vend1#"
+F 6 "C21190" H 4950 2600 50  0001 C CNN "LCSC"
 	1    4950 2600
-	1    0    0    -1
+	-1   0    0    1
 $EndComp
 $Comp
@@
 AR Path="/5E2D1A0F/5E2C1564" Ref="D23"  Part="1"
 AR Path="/5E2B6330/5E2C1564" Ref="D29"  Part="1"
-F 0 "D9" V 4989 1133 50  0000 R CNN
+F 0 "D11" V 4989 1133 50  0000 R CNN
 F 1 "LED" V 4898 1133 50  0000 R CNN
 F 2 "LED_SMD:LED_0603_1608Metric" H 4950 1250 50  0001 C CNN
@@
 F 4 "DIALIGHT,598-8010-107F" H 4950 1250 50  0001 C CNN "MFG,MFG#"
 F 5 "DIGI,350-2029-1-ND" H 4950 1250 50  0001 C CNN "Vend1,Vend1#"
+F 6 "C2286" V 4950 1250 50  0001 C CNN "LCSC"
 	1    4950 1250
 	0    -1   -1   0
@@
 AR Path="/5E2D1A0F/5E2C1FBA" Ref="R35"  Part="1"
 AR Path="/5E2B6330/5E2C1FBA" Ref="R43"  Part="1"
-F 0 "R17" H 4880 904 50  0000 R CNN
+F 0 "R19" H 4880 904 50  0000 R CNN
 F 1 "1k" H 4880 995 50  0000 R CNN
 F 2 "Resistor_SMD:R_0603_1608Metric" V 4880 950 50  0001 C CNN
@@
 F 4 "YAGEO,RC0603JR-071KL" H 4950 950 50  0001 C CNN "MFG,MFG#"
 F 5 "DIGI,311-1.0KGRCT-ND" H 4950 950 50  0001 C CNN "Vend1,Vend1#"
+F 6 "C21190" H 4950 950 50  0001 C CNN "LCSC"
 	1    4950 950
 	-1   0    0    1
@@
 AR Path="/5E2D1A0F/5E2C2529" Ref="#PWR0172"  Part="1"
 AR Path="/5E2B6330/5E2C2529" Ref="#PWR0186"  Part="1"
-F 0 "#PWR0146" H 4950 650 50  0001 C CNN
+F 0 "#PWR0148" H 4950 650 50  0001 C CNN
 F 1 "+12V" H 4965 973 50  0000 C CNN
 F 2 "" H 4950 800 50  0001 C CNN

Commit message: more available part number
Parts:
- U1: LCSC C222209 -> C377942
Changed lines of the file:
@@
 F 4 "ST,VNLD5090TR-E" H 3100 1900 50  0001 C CNN "MFG,MFG#"
 F 5 "DIGI,497-14323-1-ND" H 3100 1900 50  0001 C CNN "Vend1,Vend1#"
-F 6 "C222209" H 3100 1900 50  0001 C CNN "LCSC"
+F 6 "C377942" H 3100 1900 50  0001 C CNN "LCSC"
 	1    3100 1900
 	1    0    0    -1
